File: pcb/EtherCATControllerV1/Encoders.kicad_sch (KiCad schematic)
At the start: 8 parts, among them U5 AS5047P-ATSM

Commit message: Initial design without Ethernet connectors
Connections:
- net M0_ENC_A is gone; now on net ENC_A: C47.1, R27.2
- net M0_ENC_B is gone; now on net ENC_B: C48.1, R28.2
- net M0_ENC_Z is gone; now on net ENC_Z: C49.1, R29.2
Changed lines of the file:
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@@
 		)
 	)
-	(label "M0_ENC_B"
+	(label "ENC_B"
 		(at 205.74 57.15 0)
 		(fields_autoplaced yes)
@@
 		)
 	)
-	(label "M0_ENC_Z"
+	(label "ENC_Z"
 		(at 205.74 59.69 0)
 		(fields_autoplaced yes)
@@
 		)
 	)
-	(label "M0_ENC_A"
+	(label "ENC_A"
 		(at 205.74 54.61 0)
 		(fields_autoplaced yes)

Commit message: Added IO Board project
Other:
- note added: "Off-Axis Encoder separate Ideally through SPI TBD"
- note removed: "Off-Axis Encoder separate Ideally through SPI"
Changed lines of the file:
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@@
 		)
 	)
-	(text "Off-Axis Encoder separate\nIdeally through SPI"
+	(text "Off-Axis Encoder separate\nIdeally through SPI\nTBD"
 		(exclude_from_sim no)
-		(at 81.788 87.884 0)
+		(at 82.042 83.82 0)
 		(effects
 			(font
@@
 		(dnp no)
 		(property "Reference" "R28"
-			(at 197.104 37.846 0)
+			(at 197.358 44.958 0)
 			(effects
 				(font
@@
 		)
 		(property "Value" "3.3k"
-			(at 197.104 40.386 0)
+			(at 197.358 47.498 0)
 			(effects
 				(font
@@
 		(dnp no)
 		(property "Reference" "R29"
-			(at 204.724 37.846 0)
+			(at 205.232 44.704 0)
 			(effects
 				(font
@@
 		)
 		(property "Value" "3.3k"
-			(at 204.724 40.386 0)
+			(at 205.232 47.244 0)
 			(effects
 				(font
@@
 		(dnp no)
 		(property "Reference" "R27"
-			(at 189.484 37.846 0)
+			(at 189.738 44.958 0)
 			(effects
 				(font
@@
 		)
 		(property "Value" "3.3k"
-			(at 189.484 40.386 0)
-			(effects
-				(font
+			(at 189.738 47.498 0)
+			(effects
+				(font

Commit message: schematic finished, need to set proper ERCs
Connections:
- net VCC is gone; now on net AVCC: R27.1, R28.1, R29.1
Changed lines of the file:
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@@
 			)
 		)
-		(property "Value" "VCC"
+		(property "Value" "AVCC"
 			(at 195.326 32.766 0)
 			(effects

Commit message: Added more BOM items
Parts:
- U5: LCSC Part Number (none) -> C962063
Changed lines of the file:
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@@
+			)
+		)
+		(property "LCSC Part Number" "C962063"
+			(at 81.28 53.34 0)
+			(effects
+				(font
+					(size 1.27 1.27)
+				)
+				(hide yes)
 			)
 		)
