File: pcb/Low-Profile/EtherCATControllerLP/MOSFETs.kicad_sch (KiCad schematic)
At the start: 13 parts

Commit message: checkpoint
Parts:
- Q1: footprint DFN_2NLT1G_ONS -> (none); LCSC Part # (none) -> C348543; LCSC Part Number C348543 -> (none)
- Q10, Q2, Q5, Q6, Q9: footprint DFN_2NLT1G_ONS -> (none)
- R15, R16, R17, R18, R20, R21: LCSC Part # (none) -> C112307
- R6: LCSC Part # (none) -> C500733
Other:
- note added: "MOSFETS: NTMFS5C612NLT1G 60V, 36A Ta Downsized for low-power variant"
- note removed: "MOSFETS: NTMFS5C612NLT1G 60V, 36A Ta Downsize for low-power variant"
Changed lines of the file:
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@@
 	)
 	(junction
-		(at 130.81 139.7)
+		(at 85.09 76.2)
 		(diameter 0)
 		(color 0 0 0 0)
 	)
 	(junction
-		(at 85.09 76.2)
+		(at 179.07 76.2)
 		(diameter 0)
 		(color 0 0 0 0)
 	)
 	(junction
-		(at 179.07 76.2)
+		(at 130.81 45.72)
 		(diameter 0)
 		(color 0 0 0 0)
@@
 	)
 	(junction
-		(at 130.81 45.72)
+		(at 130.81 137.16)
 		(diameter 0)
 		(color 0 0 0 0)
 	)
 	(junction
-		(at 130.81 137.16)
+		(at 130.81 140.97)
 		(diameter 0)
 		(color 0 0 0 0)
@@
 	(wire
 		(pts
-			(xy 130.81 139.7) (xy 130.81 143.51)
+			(xy 130.81 137.16) (xy 130.81 140.97)
 		)
 		(stroke
@@
 	(wire
 		(pts
-			(xy 130.81 154.94) (xy 130.81 153.67)
+			(xy 128.27 60.96) (xy 118.11 60.96)
 		)
 		(stroke
@@
 	(wire
 		(pts
-			(xy 128.27 60.96) (xy 118.11 60.96)
+			(xy 179.07 101.6) (xy 176.53 101.6)
 		)
 		(stroke
@@
 	(wire
 		(pts
-			(xy 179.07 101.6) (xy 176.53 101.6)
+			(xy 130.81 140.97) (xy 147.32 140.97)
 		)
 		(stroke
@@
 	(wire
 		(pts
-			(xy 90.17 101.6) (xy 87.63 101.6)
+			(xy 130.81 151.13) (xy 130.81 153.67)
+		)
+		(stroke
+			(width 0)
+			(type default)
+		)
+	)
+	(wire
+		(pts
+			(xy 93.98 101.6) (xy 87.63 101.6)
 		)
 		(stroke
@@
 	(wire
 		(pts
-			(xy 130.81 153.67) (xy 130.81 151.13)
-		)
-		(stroke
-			(width 0)
-			(type default)
-		)
-	)
-	(wire
-		(pts
 			(xy 87.63 101.6) (xy 85.09 101.6)
 		)
@@
 	(wire
 		(pts
-			(xy 130.81 76.2) (xy 130.81 83.82)
+			(xy 130.81 140.97) (xy 130.81 143.51)
 		)
 		(stroke
@@
 	(wire
 		(pts
-			(xy 85.09 76.2) (xy 82.55 76.2)
+			(xy 130.81 76.2) (xy 130.81 83.82)
 		)
 		(stroke
@@
 	(wire
 		(pts
-			(xy 130.81 139.7) (xy 142.24 139.7)
+			(xy 85.09 76.2) (xy 82.55 76.2)
 		)
 		(stroke
@@
 	(wire
 		(pts
-			(xy 130.81 137.16) (xy 162.56 137.16)
+			(xy 130.81 153.67) (xy 130.81 154.94)
 		)
 		(stroke
@@
 	(wire
 		(pts
-			(xy 168.91 55.88) (xy 173.99 55.88)
+			(xy 130.81 137.16) (xy 162.56 137.16)
 		)
 		(stroke
@@
 	(wire
 		(pts
-			(xy 80.01 106.68) (xy 80.01 111.76)
+			(xy 168.91 55.88) (xy 173.99 55.88)
 		)
 		(stroke
@@
 	(wire
 		(pts
-			(xy 59.69 55.88) (xy 69.85 55.88)
+			(xy 80.01 106.68) (xy 80.01 111.76)
 		)
 		(stroke
@@
 	(wire
 		(pts
-			(xy 73.66 60.96) (xy 73.66 71.12)
+			(xy 59.69 55.88) (xy 69.85 55.88)
 		)
 		(stroke
@@
 	(wire
 		(pts
-			(xy 77.47 55.88) (xy 82.55 55.88)
+			(xy 73.66 60.96) (xy 73.66 71.12)
 		)
 		(stroke
@@
 	(wire
 		(pts
-			(xy 73.66 71.12) (xy 77.47 71.12)
+			(xy 77.47 55.88) (xy 82.55 55.88)
 		)
 		(stroke
@@
 	(wire
 		(pts
-			(xy 130.81 153.67) (xy 142.24 153.67)
+			(xy 73.66 71.12) (xy 77.47 71.12)
 		)
 		(stroke
@@
 	(wire
 		(pts
-			(xy 130.81 137.16) (xy 130.81 139.7)
+			(xy 85.09 81.28) (xy 85.09 88.9)
 		)
 		(stroke
@@
 	(wire
 		(pts
-			(xy 85.09 81.28) (xy 85.09 88.9)
+			(xy 176.53 76.2) (xy 173.99 76.2)
 		)
 		(stroke
@@
 	(wire
 		(pts
-			(xy 176.53 76.2) (xy 173.99 76.2)
+			(xy 168.91 96.52) (xy 168.91 106.68)
 		)
 		(stroke
@@
 	(wire
 		(pts
-			(xy 168.91 96.52) (xy 168.91 106.68)
+			(xy 85.09 63.5) (xy 85.09 45.72)
 		)
 		(stroke
@@
 	(wire
 		(pts
-			(xy 85.09 63.5) (xy 85.09 45.72)
+			(xy 130.81 153.67) (xy 147.32 153.67)
 		)
 		(stroke
@@
 		)
 	)
-	(text "MOSFETS: NTMFS5C612NLT1G\n60V, 36A Ta\nDownsize for low-power variant"
+	(text "MOSFETS: NTMFS5C612NLT1G\n60V, 36A Ta\nDownsized for low-power variant"
 		(exclude_from_sim no)
 		(at 106.426 87.884 0)
@@
 	)
 	(label "SL_A"
-		(at 90.17 101.6 0)
+		(at 93.98 101.6 0)
 		(fields_autoplaced yes)
 		(effects
@@
 	(hierarchical_label "SENSE_N"
 		(shape output)
-		(at 142.24 153.67 0)
+		(at 147.32 153.67 0)
 		(fields_autoplaced yes)
 		(effects
@@
 	(hierarchical_label "SENSE_P"
 		(shape output)
-		(at 142.24 139.7 0)
+		(at 147.32 140.97 0)
 		(fields_autoplaced yes)
 		(effects
@@
 			)
 		)
-		(property "Footprint" "DFN_2NLT1G_ONS"
+		(property "Footprint" ""
 			(at 77.47 71.12 0)
 			(effects
@@
 			)
 		)
-		(property "LCSC Part Number" "C348543"
+		(property "LCSC Part #" "C348543"
 			(at 77.47 71.12 0)
 			(effects
@@
 			)
 		)
+		(property "LCSC Part #" "C112307"
+			(at 165.1 111.76 0)
+			(effects
+				(font
+					(size 1.27 1.27)
+				)
+				(hide yes)
+			)
+		)
 		(pin "2"
 		)
@@
 			)
 		)
+		(property "LCSC Part #" "C500733 "
+			(at 130.81 147.32 0)
+			(effects
+				(font
+					(size 1.27 1.27)
+				)
+				(hide yes)
+			)
+		)
 		(pin "1"
 		)
@@
 			)
 		)
+		(property "LCSC Part #" "C112307"
+			(at 165.1 55.88 0)
+			(effects
+				(font
+					(size 1.27 1.27)
+				)
+				(hide yes)
+			)
+		)
 		(pin "2"
 		)
@@
 			)
 		)
+		(property "LCSC Part #" "C112307"
+			(at 73.66 55.88 0)
+			(effects
+				(font
+					(size 1.27 1.27)
+				)
+				(hide yes)
+			)
+		)
 		(pin "1"
 		)
@@
 			)
 		)
+		(property "LCSC Part #" "C112307"
+			(at 119.38 55.88 0)
+			(effects
+				(font
+					(size 1.27 1.27)
+				)
+				(hide yes)
+			)
+		)
 		(pin "2"
 		)
@@
 			)
 		)
-		(property "Footprint" "DFN_2NLT1G_ONS"
+		(property "Footprint" ""
 			(at 123.19 71.12 0)
 			(effects
@@
 			)
 		)
+		(property "LCSC Part #" "C112307"
+			(at 73.66 111.76 0)
+			(effects
+				(font
+					(size 1.27 1.27)
+				)
+				(hide yes)
+			)
+		)
 		(pin "1"
 		)
@@
 			)
 		)
+		(property "LCSC Part #" "C112307"
+			(at 118.11 111.76 0)
+			(effects
+				(font
+					(size 1.27 1.27)
+				)
+				(hide yes)
+			)
+		)
 		(pin "2"
 		)
@@
 			)
 		)
-		(property "Footprint" "DFN_2NLT1G_ONS"
+		(property "Footprint" ""
 			(at 123.19 96.52 0)
 			(effects
@@
 			)
 		)
-		(property "Footprint" "DFN_2NLT1G_ONS"
+		(property "Footprint" ""
 			(at 168.91 71.12 0)
 			(effects
@@
 			)
 		)
-		(property "Footprint" "DFN_2NLT1G_ONS"
+		(property "Footprint" ""
 			(at 168.91 96.52 0)
 			(effects
@@
 			)
 		)
-		(property "Footprint" "DFN_2NLT1G_ONS"
+		(property "Footprint" ""
 			(at 77.47 96.52 0)
 			(effects
@@
 			)
 		)
-		(property "LCSC Part Number" ""
+		(property "LCSC Part #" ""
 			(at 77.47 96.52 0)
 			(effects
