File: pcb/Low-Profile/EtherCATControllerLP/Encoders.kicad_sch (KiCad schematic)
At the start: 8 parts, among them U5 AS5047P-ATSM

Commit message: checkpoint
Parts:
- C19: LCSC Part # (none) -> C77055
- C47, C48, C49: LCSC Part # (none) -> C1532
- R27, R28, R29: LCSC Part # (none) -> C108078
- U5: LCSC Part # (none) -> C962063; LCSC Part Number C962063 -> (none)
Changed lines of the file:
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@@
+			)
+		)
+		(property "LCSC Part #" " C108078"
+			(at 195.58 45.72 0)
+			(effects
+				(font
+					(size 1.27 1.27)
+				)
+				(hide yes)
 			)
 		)
@@
 			)
 		)
+		(property "LCSC Part #" "C1532"
+			(at 163.83 63.5 0)
+			(effects
+				(font
+					(size 1.27 1.27)
+				)
+				(hide yes)
+			)
+		)
 		(pin "2"
 		)
@@
 			)
 		)
+		(property "LCSC Part #" " C108078"
+			(at 203.2 45.72 0)
+			(effects
+				(font
+					(size 1.27 1.27)
+				)
+				(hide yes)
+			)
+		)
 		(pin "1"
 		)
@@
 				)
 				(justify left bottom)
+				(hide yes)
+			)
+		)
+		(property "LCSC Part #" " C108078"
+			(at 187.96 45.72 0)
+			(effects
+				(font
+					(size 1.27 1.27)
+				)
 				(hide yes)
 			)
@@
 			)
 		)
+		(property "LCSC Part #" "C1532"
+			(at 173.99 63.5 0)
+			(effects
+				(font
+					(size 1.27 1.27)
+				)
+				(hide yes)
+			)
+		)
 		(pin "2"
 		)
@@
 			)
 		)
+		(property "LCSC Part #" "C1532"
+			(at 182.88 63.5 0)
+			(effects
+				(font
+					(size 1.27 1.27)
+				)
+				(hide yes)
+			)
+		)
 		(pin "2"
 		)
@@
 			)
 		)
-		(property "LCSC Part Number" "C962063"
+		(property "LCSC Part #" "C962063"
 			(at 81.28 53.34 0)
 			(effects
@@
 			(at 123.19 43.18 0)
 			(effects
+				(font
+					(size 1.27 1.27)
+				)
+				(hide yes)
+			)
+		)
+		(property "LCSC Part #" "C77055"
+			(at 123.19 43.18 0)
+			(effects

Commit message: Checkpoint changes before switching to XMC4800
Parts:
- C19: value 100nF -> 0.1uF
Changed lines of the file:
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@@
 			)
 		)
-		(property "Value" "100nF"
+		(property "Value" "0.1uF"
 			(at 127 44.4499 0)
 			(effects
