File: pcb/Low-Profile/IOBoard/IOBoard.kicad_sch (KiCad schematic)
At the start: 11 parts, among them J1 XT30PW-M, J3 Mounting holes, J4 DNP, J6 FH41-40S-0.5SH_05_

Commit message: Finished new 2+2 IOboard
Parts:
- removed J1: XT30PW-M, Connector_AMASS:AMASS_XT30PW-M_1x02_P2.50mm_Horizontal, symbol 2024-07-02_21-14-47:XT60PW-M
- removed J3: Mounting holes, holes:Dual Post, symbol Connector:Conn_01x02_Socket
- added J1: UMPS-02-03.5-G-V-S-W-TR, UMPS:SAMTEC_UMPS-02-03.5-G-V-S-W-TR, symbol Connector:UMPS-02-03.5-G-V-S-W-TR
- added U1: ~, Connector_AMASS:CONN-TH_4P-XT30PW-M, symbol XT302+2:XT30(2+2)PW-M.G.B
Connections:
- net SHIELD is gone; now on net GND: J6.41 (GND), J6.42 (GND), J6.43 (GND), J6.44 (GND), J6.45 (GND), J6.46 (GND), J6.47 (GND), J6.48 (GND), J6.49 (GND), J6.50 (GND)
- net DCBUS: now also J1.01, U1.1
- net ETH0_CT1: now also J6.24; no longer J6.33
- net ETH0_RX_N: now also J6.30; no longer J6.24
- net ETH0_RX_P: now also J6.28; no longer J6.22
- net ETH0_TX_N: now also J6.18; no longer J6.16
- net ETH0_TX_P: now also J6.16; no longer J6.14
- net ETH1_CT1: now also J6.22; no longer J6.36
- net ETH1_RX_N: now also J6.4; no longer J6.8
- net ETH1_RX_P: now also J6.6; no longer J6.10
- net ETH1_TX_N: now also J6.32; no longer J6.28
- net ETH1_TX_P: now also J6.34; no longer J6.30
- net GND: now also J6.10, J6.14, J6.33, J6.36, J6.8, J1.02, U1.2; no longer J6.18, J6.32, J6.34, J6.37, J6.39, J6.4, J6.6
- new net CAN_H: J6.37, U1.3
- new net CAN_L: J6.39, U1.4
Other:
- note added: "Note: LP one uses XT30(2+2) HP one uses XT60"
- note added: "Power connectors using Samtec UMPT-02/UMPS-02"
- note removed: "Note: LP one uses XT30"
- note removed: "Power Connectors: Molex 2032631334 (Male) 2043180018 (Female)"

Commit message: Added XMC4800
Other:
- note added: "ETH1 optional for Line Topology Shared cable with 4 pairs hosts both in and out"
Changed lines of the file:
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@@
+		)
+	)
+	(text "ETH1 optional for Line Topology\nShared cable with 4 pairs hosts\nboth in and out"
+		(exclude_from_sim no)
+		(at 158.242 153.924 0)
+		(effects
+			(font
+				(size 1.27 1.27)
+			)
 		)
 	)
