File: pcb/low-power/EtherCATSTM32/Connectors.kicad_sch (KiCad schematic)
At the start: 22 parts, among them J1 FH41-40S-0.5SH_05_, J2 Conn_01x02_Socket, J3 Conn_01x04_Socket, J4 TYPE-C-31-M-12, J5 Mounting holes, J6 Conn_01x03_Pin, SW1 EVP-AA202K

Commit message: starting HP version
Parts:
- removed J2: Conn_01x02_Socket, Connector_PinHeader_1.00mm:PinHeader_1x02_P1.00mm_Vertical, symbol Connector:Conn_01x02_Socket
- removed J5: Mounting holes, UMPT:SAMTEC_UMPT-02-12.5-X-V-S-W-X, symbol Connector:Conn_01x02_Socket
- removed J6: Conn_01x03_Pin, Connector_PinHeader_1.00mm:PinHeader_1x03_P1.00mm_Vertical, symbol Connector:Conn_01x03_Pin
- added J2: Right Angle 1x4, Connector_PinHeader_1.00mm:PinHeader_1x04_P1.00mm_Vertical, symbol Connector:Conn_01x04_Pin
- added J5: UMPT-02-12.5-X-V-S-W-X, UMPT:SAMTEC_UMPT-02-12.5-X-V-S-W-X, symbol samtec:UMPT-02-12.5-X-V-S-W-X
- added R41, R42: 22R, Resistor_SMD:R_0603_1608Metric, symbol Device:R
- H7, H8, H9: footprint Connector_PinHeader_2.54mm:PinHeader_1x01_P2.54mm_Vertical -> MountingHole:MountingHole_2.2mm_M2_Pad
- J1: footprint Connector_FFC-FPC:Hirose_FH41-30S-0.5SH_1x30_1MP_1SH_P0.5mm_Horizontal -> FH41:HRS_FH41-40S-0.5SH_05_
- J3: now not fitted
- J4: footprint Connector_USB:USB_C_Receptacle_HRO_TYPE-C-31-M-12 -> footprints:HRO_TYPE-C-31-M-12
Connections:
- net DCBUS: now also J5.01
- net GND: now also J2.2 (Pin_2), J5.02
- net VCC: now also J2.4 (Pin_4)
- net RESET renamed BOOT0
- net VBUS_USB: no longer names the net of J4.A4_B9 (VBUS), J4.B4_A9 (VBUS)
- new net: J2.1 (Pin_1), R42.2
- new net: J2.3 (Pin_3), R41.1
- new net SWCLK: R41.2
- new net SWDIO: R42.1
- no-connect marks 4 -> 5
Other:
- note added: "SW Debug"
