File: pcb/low-power/EtherCATSTM32/Encoders.kicad_sch (KiCad schematic)
At the start: 8 parts, among them U5 AS5047P-ATSM

Commit message: starting HP version
Parts:
- removed C47, C48, C49: 22nF, Capacitor_SMD:C_0402_1005Metric, symbol Device:C
- removed R27, R28, R29: 3.3k, Resistor_SMD:R_0603_1608Metric, symbol Device:R
Other:
- moved on the sheet: C19, U5
