File: pcb/low-power/EtherCATSTM32/EtherCAT.kicad_sch (KiCad schematic)
At the start: 45 parts, among them U4 LAN9252I/ML, U7 24FC512-I/SN, Y2 ABM8-25.000MHZ-D2Y-T

Commit message: starting HP version
Parts:
- removed R10, R19, R22, R26, R30, R32: 49.9, symbol Device:R_Small
- removed R34: 0, symbol Device:R_Small
- removed R40: 2k, symbol Device:R_Small
- added RN1, RN2: 49R9, Resistor_SMD:R_Array_Convex_4x0402, symbol Device:R_Pack04_Split
- C36: footprint 0603 -> Capacitor_SMD:C_0603_1608Metric
- C38, C39: footprint (none) -> Capacitor_SMD:C_0402_1005Metric; LCSC Part # (none) -> C76701
- C50, C53, C55, C57, C58, C70, C73, C75: footprint (none) -> Capacitor_SMD:C_0603_1608Metric; LCSC Part # (none) -> C77055
- C51, C52: footprint (none) -> Capacitor_SMD:C_0603_1608Metric; LCSC Part # (none) -> C106858
- C54: footprint (none) -> Capacitor_SMD:C_0402_1005Metric; LCSC Part # (none) -> C106207
- C59, C60, C61, C63, C64, C65, C66, C67: footprint (none) -> Capacitor_SMD:C_0402_1005Metric; LCSC Part # (none) -> C115606
- C68, C69: footprint (none) -> Capacitor_SMD:C_0402_1005Metric; LCSC Part # (none) -> C147616
- FB1, FB2, FB3, FB4: footprint (none) -> Inductor_SMD:L_1206_3216Metric
- R33: footprint (none) -> Resistor_SMD:R_0402_1005Metric; LCSC Part # (none) -> C106231
- R35: footprint (none) -> Resistor_SMD:R_0402_1005Metric; LCSC Part # (none) -> C105871
- R36: footprint (none) -> Resistor_SMD:R_0402_1005Metric; LCSC Part # (none) -> C281773
- R37: footprint (none) -> Resistor_SMD:R_0402_1005Metric; LCSC Part # (none) -> C144035
- R8: value 49.9 -> 2k; footprint (none) -> Resistor_SMD:R_0402_1005Metric; LCSC Part # (none) -> C144035
- R9: value 49.9 -> 0; footprint (none) -> Resistor_SMD:R_0402_1005Metric; LCSC Part # (none) -> C106231
- U4: footprint (none) -> footprints:QFN64_ML_MCH
- U7: footprint (none) -> Package_SO:SOP-8_3.9x4.9mm_P1.27mm
- Y2: footprint (none) -> Crystal:Crystal_SMD_3225-4Pin_3.2x2.5mm
Connections:
- net ETH0_RXN: now also U4.61 (RXNB), RN1.2 (R2.1); no longer U4.54 (RXNA)
- net ETH0_RXP: now also U4.60 (RXPB), RN1.1 (R1.1); no longer R8.2, U4.55 (RXPA)
- net ETH0_TXN: now also U4.63 (TXNB), RN1.4 (R4.1); no longer U4.52 (TXNA)
- net ETH0_TXP: now also U4.62 (TXPB), RN1.3 (R3.1); no longer U4.53 (TXPA)
- net ETH1_CT1: now also R9.2
- net ETH1_RXN: now also U4.54 (RXNA), RN2.3 (R3.1); no longer U4.61 (RXNB)
- net ETH1_RXP: now also U4.55 (RXPA), RN2.4 (R4.1); no longer U4.60 (RXPB)
- net ETH1_TXN: now also U4.52 (TXNA), RN2.1 (R1.1); no longer R9.2, U4.63 (TXNB)
- net ETH1_TXP: now also U4.53 (TXPA), RN2.2 (R2.1); no longer U4.62 (TXPB)
- net EtherCAT3v3: now also R8.1; no longer U4.42 (EESDA/TMS), U7.5 (SDA)
- net VDDTXRX1: now also RN1.5 (R4.2), RN1.6 (R3.2), RN1.7 (R2.2), RN1.8 (R1.2); no longer R8.1
- net VDDTXRX2: now also RN2.5 (R4.2), RN2.6 (R3.2), RN2.7 (R2.2), RN2.8 (R1.2)
- new net I2C_SDA: R8.2, U4.42 (EESDA/TMS), U7.5 (SDA)
