File: pcb/low-power/EtherCATSTM32/EtherCATSTM32.kicad_pcb (KiCad board)
At the start: 6 copper layers, 50 x 50 mm, 178 parts, among them J1 FH41-40S-0.5SH_05_, J2 Conn_01x02_Socket, J3 Conn_01x04_Socket, J4 TYPE-C-31-M-12, J5 Mounting holes, J6 Conn_01x03_Pin, SW1 EVP-AA202K, U1 DP83849IFVS_NOPB, U2 TPS54360DDAR, U3 LDL1117S33R, U4 NC7SZ125P5X, U5 AS5047P-ATSM, U6 MCF8329A1IREER, U8 SN65HVD231, Y1 32.768 KHZ, Y2 12 MHz

Commit message: starting HP version
Parts:
- removed C11: 0.1uF, Capacitor_SMD:C_0603_1608Metric
- removed C30, C31, C37, C56: 10uF, Capacitor_SMD:C_0805_2012Metric
- removed C47, C48, C49: 22nF, Capacitor_SMD:C_0402_1005Metric
- removed FB6: BLM18PG600, Inductor_SMD:L_0603_1608Metric
- removed J6: Conn_01x03_Pin, Connector_PinHeader_1.00mm:PinHeader_1x03_P1.00mm_Vertical
- removed R10, R22: 2.2K, Resistor_SMD:R_0402_1005Metric
- removed R26, R30: 10k, Resistor_SMD:R_0603_1608Metric
- removed R27, R28, R29: 3.3k, Resistor_SMD:R_0603_1608Metric
- removed RN3, RN4, RN5, RN6, RN7: 49R9, Resistor_THT:R_Array_SIP5
- added C73: 0.1uF, Capacitor_SMD:C_0603_1608Metric, F.Cu at (152.8, 85.8)
- added C75: 0.1uF, Capacitor_SMD:C_0603_1608Metric, F.Cu at (140.2, 79.0)
- added C76: 1uF, Capacitor_SMD:C_0603_1608Metric, F.Cu at (163.8, 91.6)
- added C77: 0.1uF, Capacitor_SMD:C_0603_1608Metric, F.Cu at (163.8, 90.0)
- added FB2: 2A, 0.05DCR, Inductor_SMD:L_1206_3216Metric, F.Cu at (144.4, 87.6)
- added FB3: 2A, 0.05DCR, Inductor_SMD:L_1206_3216Metric, F.Cu at (142.6, 97.2)
- added R33: 0, Resistor_SMD:R_0402_1005Metric, F.Cu at (139.0, 100.6)
- added R35: 4.7k, Resistor_SMD:R_0402_1005Metric, F.Cu at (138.6, 79.6)
- added R36: 12.1K, Resistor_SMD:R_0402_1005Metric, F.Cu at (145.8, 102.2)
- added R37: 2k, Resistor_SMD:R_0402_1005Metric, F.Cu at (145.8, 84.8)
- added R41: 22R, Resistor_SMD:R_0603_1608Metric, F.Cu at (162.4, 84.2)
- added R42: 22R, Resistor_SMD:R_0603_1608Metric, F.Cu at (160.8, 84.2)
- C1, C10, C2, C3, C4, C5, C6, C9: footprint Capacitor_SMD:C_2220_5750Metric -> Capacitor_SMD:C_1210_3225Metric; moved to B.Cu
- C12, C14, C15, C18, C19, C20, C21, C22, C23, C24, C25, C26, C28, C29, C40, C42, C43, C44, C45, C46, C62, C72, C74, C82, C84, D2, L1, R1, R11, R12, R13, R14, R2, R25, R3, R38, R39, R4, R44, R45, R46, R47, R50, R52, R6, TH3, U2, U8: moved to B.Cu
- C13, C33: value 0.1uF -> 10pF; footprint Capacitor_SMD:C_0603_1608Metric -> Capacitor_SMD:C_0402_1005Metric; moved to B.Cu
- C34, C35: value 0.1uF -> 2.2µF
- C36, C51, C52: value 0.1uF -> 1uF
- C38, C39: value 15pF -> 18pF
- C54: value 10uF -> 470pF
- C59, C60, C61, C63, C65, C66, C67: value 0.1uF -> 10pF; footprint Capacitor_SMD:C_0603_1608Metric -> Capacitor_SMD:C_0402_1005Metric
- C64: value 10uF -> 10pF; footprint Capacitor_SMD:CP_Elec_6.3x5.4 -> Capacitor_SMD:C_0402_1005Metric
- C68, C69: value 0.1uF -> 0.022uF; footprint Capacitor_SMD:C_0603_1608Metric -> Capacitor_SMD:C_0402_1005Metric
- C7, C8: value 22uF -> 10uF; footprint Capacitor_SMD:C_2220_5750Metric -> Capacitor_SMD:C_1210_3225Metric; moved to B.Cu
- FB1, FB4, FB5: value BLM18PG600 -> 2A, 0.05DCR; footprint Inductor_SMD:L_0603_1608Metric -> Inductor_SMD:L_1206_3216Metric
- H7, H8, H9: footprint Connector_PinHeader_2.54mm:PinHeader_1x01_P2.54mm_Vertical -> MountingHole:MountingHole_2.2mm_M2_Pad
- J1: footprint Connector_FFC-FPC:Hirose_FH41-30S-0.5SH_1x30_1MP_1SH_P0.5mm_Horizontal -> FH41:HRS_FH41-40S-0.5SH_05_
- J2: value Conn_01x02_Socket -> Right Angle 1x4; footprint Connector_PinHeader_1.00mm:PinHeader_1x02_P1.00mm_Vertical -> Connector_PinHeader_1.00mm:PinHeader_1x04_P1.00mm_Vertical
- J4: footprint Connector_USB:USB_C_Receptacle_HRO_TYPE-C-31-M-12 -> footprints:HRO_TYPE-C-31-M-12
- J5: value Mounting holes -> UMPT-02-12.5-X-V-S-W-X
- R7: value 510R -> 47K
- R8: value 1.5K -> 2k
- R9: value 4.87k, 1% -> 0; footprint Resistor_SMD:R_0603_1608Metric -> Resistor_SMD:R_0402_1005Metric
- RN1, RN2: footprint Resistor_THT:R_Array_SIP5 -> Resistor_SMD:R_Array_Convex_4x0402
- U1: value DP83849IFVS_NOPB -> STM32F405RGT6; footprint DP83849:QFP50P1400X1400X120-80N -> Package_QFP:LQFP-64_10x10mm_P0.5mm; moved to B.Cu
- U4: value NC7SZ125P5X -> LAN9252I/ML; footprint Package_TO_SOT_SMD:SOT-353_SC-70-5 -> footprints:QFN64_ML_MCH
- U7: value ~ -> 24FC512-I/SN; footprint XMC4800:LQFP-100-XMC4800 -> Package_SO:SOP-8_3.9x4.9mm_P1.27mm
- Y1: value 32.768 KHZ -> ABM3B-8.000MHZ-10-1-U-T; footprint Crystal:Crystal_SMD_3215-2Pin_3.2x1.5mm -> Crystal:Crystal_SMD_5032-4Pin_5.0x3.2mm; moved to B.Cu
- Y2: value 12 MHz -> ABM8-25.000MHZ-D2Y-T
- moved C42 135.1 mm to (173.2, 99.6), turned to 180 degrees
- moved RN1 134.5 mm to (138.4, 98.3), turned to -90 degrees
- moved C5 133.6 mm to (158.6, 114.8), turned to -90 degrees
- moved C36 133.2 mm to (160.6, 93.2)
- moved C40 132.7 mm to (171.2, 93.0)
- moved C33 132.6 mm to (160.0, 85.4)
- moved R23 132.4 mm to (173.4, 103.8), turned to 90 degrees
- moved C4 131.9 mm to (155.4, 114.8), turned to -90 degrees
- moved C58 131.6 mm to (160.6, 91.6)
- moved C43 131.0 mm to (171.2, 91.4)
- moved C3 130.7 mm to (152.2, 114.8), turned to -90 degrees
- moved R24 130.2 mm to (171.8, 103.8), turned to -90 degrees
- moved C2 129.9 mm to (149.0, 114.8), turned to -90 degrees
- moved RN2 129.8 mm to (138.7, 93.0), turned to 90 degrees
- moved C1 129.6 mm to (145.8, 114.8), turned to -90 degrees
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Connections:
- C13 pad 1: VCC -> Net-(U1-PH0)
- C32 pad 1: VCC -> /NRST
- C33 pad 1: VCC -> Net-(U1-PH1)
- C34 pad 1: VCC -> Net-(U1-VCAP_1)
- C35 pad 1: VCC -> Net-(U1-VCAP_2)
- C36 pad 1: VCC -> VDDCR
- C38 pad 1: /MCU/RTC_XTAL2 -> GND
- C38 pad 2: GND -> Net-(U4-OSCI)
- C39 pad 1: /MCU/RTC_XTAL1 -> GND
- C39 pad 2: GND -> Net-(U4-OSCO)
- C50 pad 1: VDDC -> VDDCR
- C51 pad 1: VDDC -> VDDTXRX1
- C52 pad 1: VDDC -> VDDTXRX2
- C53 pad 1: VDDC -> VDDBIAS
- C54 pad 1: VDDC -> VDDCR
- C55 pad 1: /MCU/VDDA -> VDDTXRX1
- C57 pad 1: /MCU/VAREF -> VDDTXRX2
- C58 pad 1: /EtherCAT/PFBOUT -> VDDCR
- C59 pad 1: /EtherCAT/PFBOUT -> /ETH0_RXP
- C60 pad 1: /EtherCAT/PFBOUT -> /ETH1_TXN
- C61 pad 1: /EtherCAT/PFBOUT -> /ETH0_RXN
- C63 pad 1: /EtherCAT/PFBOUT -> /ETH1_TXP
- C64 pad 1: /EtherCAT/PFBOUT -> /ETH0_TXP
- C65 pad 1: VCC -> /ETH1_RXN
- C66 pad 1: /EtherCAT/VCCTXRX -> /ETH0_TXN
- C67 pad 1: /EtherCAT/VCCTXRX -> /ETH1_RXP
- C68 pad 1: /EtherCAT/VCCTXRX -> /ETH0_CT1
- C69 pad 1: /ETH0_CT1 -> /ETH1_CT1
- C70 pad 1: /ETH1_CT1 -> Net-(U4-VDD12TX1)
- C71 pad 1: /RESET -> /BOOT0
- FB1 pad 1: /EtherCAT/VCCTXRX -> EtherCAT3v3
- FB1 pad 2: VCC -> VDDTXRX1
- FB4 pad 1: /VBUS_USB -> Net-(U4-VDD12TX1)
- FB4 pad 2: Net-(U7-VBUS) -> VDDCR
- FB5 pad 1: /MCU/VAREF -> VCC
- FB5 pad 2: VCC -> EtherCAT3v3
- J2 pad 1: /UART_TX -> Net-(J2-Pin_1)
- J2 pad 2: /UART_RX -> GND
- J5 pad 01: (no net) -> DCBUS
- J5 pad 02: (no net) -> GND
- R31 pad 2: /RESET -> /BOOT0
- R7 pad 1: Net-(R7-Pad1) -> /BOOT0
- R7 pad 2: /MCU/XTAL2 -> GND
- R8 pad 1: VCC -> EtherCAT3v3
- R8 pad 2: /MDIO -> /EtherCAT/I2C_SDA
- R9 pad 1: GND -> VDDTXRX2
- R9 pad 2: Net-(U1-RBIAS) -> /ETH1_CT1
- RN1 pad 1: Net-(RN1A-R1) -> /ETH0_RXP
- RN1 pad 2: Net-(RN1B-R2.1) -> /ETH0_RXN
- RN1 pad 3: Net-(RN1C-R3.1) -> /ETH0_TXP
- RN1 pad 4: Net-(RN1D-R4.1) -> /ETH0_TXN
- RN1 pad 5: /ECAT0.P0_TXD3 -> VDDTXRX1
- RN2 pad 1: Net-(RN2A-R1) -> /ETH1_TXN
- RN2 pad 2: Net-(RN2B-R2.1) -> /ETH1_TXP
- RN2 pad 3: Net-(RN2C-R3.1) -> /ETH1_RXN
- RN2 pad 4: Net-(RN2D-R4.1) -> /ETH1_RXP
- RN2 pad 5: /ECAT0.P1_TXD1 -> VDDTXRX2
- SW1 pad 1: /RESET -> /BOOT0
- U1 pad 1: unconnected-(U1-CRS_A/CRS_DV_A/LED_CFG_A-Pad1) -> VCC
- U1 pad 10: GND -> /WAKE
- U1 pad 11: VCC -> /DRVOFF
- U1 pad 12: Net-(RN5A-R1) -> GND
- U1 pad 13: /ECAT0.P0_TX_ENA -> VCC
- U1 pad 14: Net-(RN1A-R1) -> unconnected-(U1-PA0-Pad14)
- U1 pad 15: Net-(RN1B-R2.1) -> /TEMP_BACKSIDE
- U1 pad 16: Net-(RN1C-R3.1) -> /TEMP_MOSFETS
- U1 pad 17: Net-(RN1D-R4.1) -> /TEMP_ICS
- U1 pad 18: /POWERDOWN_A -> GND
- U1 pad 19: unconnected-(U1-LED_LINK_A/AN0_A-Pad19) -> VCC
- U1 pad 2: /ECAT0_P0_RX_ERRB -> /SPI2_CS
- U1 pad 20: unconnected-(U1-LED_SPEED_A/AN1_A-Pad20) -> /VBUS_SENSE
- U1 pad 21: unconnected-(U1-LED_ACT/LED_COL/AN_EN_A-Pad21) -> /SPI_SCK
- U1 pad 22: GND -> /SPI_MISO
- U1 pad 23: /ETH0_RXN -> /SPI_MOSI
- U1 pad 24: /ETH0_RXP -> unconnected-(U1-PC4-Pad24)
- U1 pad 25: GND -> /IRQ
- U1 pad 26: /ETH0_TXN -> unconnected-(U1-PB0-Pad26)
- U1 pad 27: /ETH0_TXP -> unconnected-(U1-PB1-Pad27)
- U1 pad 28: /EtherCAT/PFBOUT -> GND
- U1 pad 29: GND -> /I2C_SDA
- U1 pad 3: /EtherCAT/COL_PHYAD0_A -> unconnected-(U1-PC14-Pad3)
- U1 pad 30: VCC -> /I2C_SCL
- U1 pad 31: /EtherCAT/PFBOUT -> Net-(U1-VCAP_1)
- U1 pad 32: Net-(U1-RBIAS) -> VCC
- U1 pad 33: GND -> /SPI1_CS
- U1 pad 34: /EtherCAT/PFBOUT -> /SPI1_SCK
- U1 pad 35: /ETH1_TXP -> /SPI1_MISO
- U1 pad 36: /ETH0_TXN -> /SPI1_MOSI
- U1 pad 37: GND -> /ETHRST
- U1 pad 38: /ETH1_RXP -> unconnected-(U1-PC7-Pad38)
- U1 pad 39: /ETH1_RXN -> unconnected-(U1-PC8-Pad39)
- U1 pad 4: Net-(RN3A-R1) -> unconnected-(U1-PC15-Pad4)
- U1 pad 40: GND -> unconnected-(U1-PC9-Pad40)
- U1 pad 41: unconnected-(U1-LED_ACT/LED_COL/AN_EN_B-Pad41) -> /SPI_CS
- U1 pad 44: /POWERDOWN_B -> /USB_D-
- U1 pad 45: Net-(RN2A-R1) -> /USB_D+
- U1 pad 46: Net-(RN2B-R2.1) -> /SWDIO
- U1 pad 47: Net-(RN2D-R4.1) -> Net-(U1-VCAP_2)
- U1 pad 48: Net-(RN2C-R3.1) -> VCC
- U1 pad 49: /ECAT0.P1_TX_ENA -> /SWCLK
- U1 pad 5: Net-(RN3B-R2.1) -> Net-(U1-PH0)
- U1 pad 50: Net-(RN5B-R2.1) -> unconnected-(U1-PA15-Pad50)
- U1 pad 51: VCC -> /SPI2_SCK
- U1 pad 52: GND -> /SPI2_MISO
- U1 pad 53: Net-(RN4D-R4.1) -> /SPI2_MOSI
- U1 pad 54: /EtherCAT/PFBOUT -> /NFAULT
- U1 pad 55: GND -> unconnected-(U1-PB3-Pad55)
- U1 pad 56: Net-(RN4C-R3.1) -> unconnected-(U1-PB4-Pad56)
- U1 pad 57: Net-(RN4B-R2.1) -> /CAN_RX
- U1 pad 58: Net-(RN4A-R1) -> /CAN_TX
- U1 pad 6: GND -> Net-(U1-PH1)
- U1 pad 60: /ECAT0.P1_RX_ERRB -> /BOOT0
- U1 pad 62: /ECAT0.P1_RX_DVA -> unconnected-(U1-PB9-Pad62)
- U1 pad 63: Net-(RN5C-R3.1) -> GND
- U1 pad 64: GND -> VCC
- U1 pad 7: /EtherCAT/PFBOUT -> /NRST
- U1 pad 8: Net-(RN3C-R3.1) -> /BRAKE
- U1 pad 9: Net-(RN3D-R4.1) -> /DIR
- U4 pad 1: GND -> Net-(U4-OSCI)
- U4 pad 2: /ECAT_RST -> Net-(U4-OSCO)
- U4 pad 3: GND -> unconnected-(U4-OSCVDD12-Pad3)
- U4 pad 4: /EtherCAT/PHY_RST -> GND
- U4 pad 5: VCC -> EtherCAT3v3
- U7 pad 1: /ECAT0.P1_RX_CLK -> /EtherCAT/WP
- U7 pad 2: /ECAT_RST -> /EtherCAT/WP
- U7 pad 3: /ECAT0.P1_TX_CLK -> /EtherCAT/WP
- U7 pad 4: unconnected-(U7-P0.9-Pad4) -> GND
- U7 pad 5: /ECAT0.P1_TXD1 -> /EtherCAT/I2C_SDA
- U7 pad 6: /ECAT0.P1_TXD0 -> /EtherCAT/I2C_SCL
- U7 pad 7: /ECAT0.P1_TX_ENA -> /EtherCAT/WP
- U7 pad 8: /USB_D- -> EtherCAT3v3
- Y1 pad 1: /MCU/RTC_XTAL2 -> Net-(U1-PH0)
- Y1 pad 2: /MCU/RTC_XTAL1 -> GND
- Y2 pad 1: /MCU/XTAL1 -> Net-(U4-OSCI)
- Y2 pad 3: Net-(R7-Pad1) -> Net-(U4-OSCO)
Routing:
- added copper zone on In2.Cu, net 5V
- added copper zone on In2.Cu, net DCBUS
- added copper zone on In2.Cu, net EtherCAT3v3
- added copper zone on In1.Cu, net GND
- added copper zone on In4.Cu, net GND
- added copper zone on In2.Cu, net VCC
