File: pcb/low-power/EtherCATSTM32/EtherCATSTM32.kicad_sch (KiCad schematic)
At the start: 0 parts

Commit message: starting HP version
Other:
- sheet Connectors ports: added BOOT0, SWCLK, SWDIO; removed RESET, SWV, TCK, TMS, UART_RX, UART_TX, VBUS_USB
- sheet EtherCAT ports: added none; removed ETH0_CT2, ETH1_CT2
- sheet MCU ports: added CAN_RX, CAN_TX; removed M0_ENC_A, M0_ENC_B, M0_ENC_Z, PGOOD
