File: pcb/low-power/EtherCATSTM32/MCU.kicad_sch (KiCad schematic)
At the start: 8 parts, among them U1 STM32F405RGT6, Y1 ABM3B-8.000MHZ-10-1-U-T

Commit message: starting HP version
Parts:
- C13, C33: footprint Capacitor_SMD:C_0603_1608Metric -> Capacitor_SMD:C_0402_1005Metric; LCSC Part # (none) -> C115606
- C32: LCSC Part # (none) -> C77055
- C34, C35: LCSC Part # (none) -> C77183
- R7: LCSC Part # (none) -> C105579
Connections:
- net AVCC is gone; now on net VCC: U1.13 (VDDA)
- net M0_ENC_A: no longer names the net of U1.56 (PB4)
- net M0_ENC_B renamed CAN_RX
- net M0_ENC_Z renamed CAN_TX
- net PGOOD: no longer names the net of U1.50 (PA15)
- no-connect marks 15 -> 17
