File: pcb/low-power/EtherCATSTM32/Power.kicad_sch (KiCad schematic)
At the start: 26 parts

Commit message: starting HP version
Parts:
- removed C11: ${CAPACITANCE}, Capacitor_SMD:C_0603_1608Metric, symbol Device:C
- removed C30, C31, C37, C56: 10uF, Capacitor_SMD:C_0805_2012Metric, symbol Device:C
- added C76: 1uF, Capacitor_SMD:C_0603_1608Metric, symbol Device:C_Small
- added C77: ${CAPACITANCE}, Capacitor_SMD:C_0603_1608Metric, symbol Device:C
- added FB5: 2A, 0.05DCR, Inductor_SMD:L_1206_3216Metric, symbol Device:FerriteBead_Small
- C1, C10, C2, C3, C4, C5, C6, C9: footprint Capacitor_SMD:C_2220_5750Metric -> Capacitor_SMD:C_1210_3225Metric; LCSC Part # C153035 -> C5156756
- C7, C8: value 22uF -> 10uF; footprint Capacitor_SMD:C_2220_5750Metric -> Capacitor_SMD:C_1210_3225Metric; LCSC Part # C1921234 -> C5156756
Connections:
- net GND: now also C76.2, C77.2
- net VCC: now also FB5.1
- new net EtherCAT3v3: C76.1, C77.1, FB5.2
