File: pcb/high-power/EtherCATControllerHP/EtherCATControllerHP.kicad_sch (KiCad schematic)
At the start: 0 parts

Commit message: starting HP version
Other:
- added sheet CAN (CAN.kicad_sch)
- added sheet Temperature Sensors (Temperature.kicad_sch)
- sheet Connectors ports: added CAN_H, CAN_L, ETH0_RX_N, ETH0_RX_P, ETH0_TX_N, ETH0_TX_P, ETH1_RX_N, ETH1_RX_P, ETH1_TX_N, ETH1_TX_P, USB_D+, USB_D-; removed ETH0_CT2, ETH0_RXN, ETH0_RXP, ETH0_TXN, ETH0_TXP, ETH1_CT2, ETH1_RXN, ETH1_RXP, ETH1_TXN, ETH1_TXP, NRST, USB_DM, USB_DP
- sheet Encoders ports: added none; removed ENC_A, ENC_B, ENC_Z
- sheet EtherCAT ports: added none; removed ETH0_CT2, ETH1_CT2
- sheet MCU ports: added CAN_RX, CAN_TX, TEMP_BACKSIDE, TEMP_ICS, TEMP_MOSFETS, USB_D+, USB_D-; removed M0_ENC_A, M0_ENC_B, M0_ENC_Z, PGOOD, USB_DM, USB_DP
- sheet Power ports: added none; removed PGOOD

Commit message: stash before via stitching
Other:
- sheet MCU ports: added CAN_MODE; removed BRAKE, DIR, TEMP_BACKSIDE, TEMP_ICS
- sheet Motor ports: added none; removed BRAKE, DIR
- sheet Temperature Sensors ports: added none; removed TEMP_BACKSIDE, TEMP_ICS
