File: pcb/high-power/EtherCATControllerHP/Regulators.kicad_sch (KiCad schematic)
At the start: 0 parts

Commit message: starting HP version
Parts:
- added C12: 4.7uF, Capacitor_SMD:C_1210_3225Metric, symbol Device:C_Small
- added C14: 0.1uF, Capacitor_SMD:C_0402_1005Metric, symbol Device:C_Small
- added C15: 6800pF, Capacitor_SMD:C_0402_1005Metric, symbol Device:C_Small
- added C16, C17: 4.7uF, Capacitor_SMD:C_0805_2012Metric, symbol Device:C
- added C18: 39pF, Capacitor_SMD:C_0402_1005Metric, symbol Device:C_Small
- added C72, C74: 47uF, Capacitor_SMD:C_0805_2012Metric, symbol Device:C_Small
- added D1: LTST-C190KGKT, Diode_SMD:D_0603_1608Metric, symbol LTST-C190KGKT:LTST-C190KGKT
- added D2: B560C, Diode_SMD:D_SMC, symbol Device:D_Schottky
- added L1: 8.2uH, Inductor_SMD:L_Sunlord_MWSA0603S, symbol Device:L_Small
- added R1: 162K, Resistor_SMD:R_0603_1608Metric, symbol Device:R_Small
- added R2: 523K, Resistor_SMD:R_0402_1005Metric, symbol Device:R_Small
- added R3: 84R5, Resistor_SMD:R_0603_1608Metric, symbol Device:R_Small
- added R38: 53.6K, Resistor_SMD:R_0603_1608Metric, symbol Device:R_Small
- added R39: 10.2K, Resistor_SMD:R_0402_1005Metric, symbol Device:R_Small
- added R4: 13K, Resistor_SMD:R_0402_1005Metric, symbol Device:R_Small
- added R5: 1k, Resistor_SMD:R_0603_1608Metric, symbol Device:R
- added TP2, TP3: TESTPOINT, TestPoint:TestPoint_Pad_1.0x1.0mm, symbol Connector:TestPoint
- added U2: TPS54360DDAR, Package_SO:TI_SO-PowerPAD-8_ThermalVias, symbol Regulator_Switching:TPS54360DDA
- added U3: LDL1117S33R, Package_TO_SOT_SMD:SOT-223, symbol LDL1117S33R:LDL1117S33R
Connections:
- new net: D1.2, R5.1, TP2.1
- new net: R2.2, R3.1
- new net: C14.1, U2.1 (BOOT)
- new net: R1.1, U2.4 (RT/CLK)
- new net: C18.1, R4.1, U2.6 (COMP)
- new net: C14.2, D2.1 (K), L1.1, U2.8 (SW)
- new net: C15.1, R4.2
- new net 5V: C72.1, C74.1, L1.2, R38.1, TP3.1, U3.3 (VIN)
- new net DCBUS: C12.1, R2.1, U2.2 (VIN)
- new net FB: R38.2, R39.1, U2.5 (FB)
- new net GND: C12.2, C15.2, C16.2, C17.2, C18.2, C72.2, C74.2, D2.2 (A), R1.2, R3.2, R39.2, R5.2, U2.3 (EN), U2.7 (GND), U2.9 (GNDPAD), U3.1 (GND)
- new net VCC: C16.1, C17.1, D1.1, U3.2 (VOUT), U3.4 (VOUT)
Other:
- note added: "3v3"
- note added: "5V out"

Commit message: stash before via stitching
Parts:
- R2: footprint Resistor_SMD:R_0402_1005Metric -> Resistor_SMD:R_0603_1608Metric_Pad0.98x0.95mm_HandSolder; LCSC Part # C327338 -> C23076
- R3: value 84R5 -> 84.5k; LCSC Part # C334834 -> C706195
Connections:
- net GND: no longer U2.3 (EN)
- net VCC: now also TP2.1
- net at D1.2, R5.1: no longer TP2.1
- net at R2.2, R3.1: now also U2.3 (EN)
Changed lines of the file:
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@@
 	)
 	(junction
-		(at 100.33 62.23)
-		(diameter 0)
-		(color 0 0 0 0)
-	)
-	(junction
-		(at 186.69 109.22)
-		(diameter 0)
-		(color 0 0 0 0)
-	)
-	(junction
 		(at 168.91 54.61)
 		(diameter 0)
@@
 	)
 	(junction
+		(at 104.14 62.23)
+		(diameter 0)
+		(color 0 0 0 0)
+	)
+	(junction
 		(at 104.14 49.53)
 		(diameter 0)
@@
 	(wire
 		(pts
-			(xy 100.33 60.96) (xy 100.33 62.23)
-		)
-		(stroke
-			(width 0)
-			(type default)
-		)
-	)
-	(wire
-		(pts
 			(xy 104.14 71.12) (xy 104.14 68.58)
 		)
@@
 	(wire
 		(pts
-			(xy 100.33 62.23) (xy 110.49 62.23)
-		)
-		(stroke
-			(width 0)
-			(type default)
-		)
-	)
-	(wire
-		(pts
 			(xy 157.48 62.23) (xy 168.91 62.23)
 		)
@@
 	(wire
 		(pts
-			(xy 100.33 62.23) (xy 100.33 71.12)
+			(xy 100.33 60.96) (xy 100.33 71.12)
 		)
 		(stroke
@@
 	(wire
 		(pts
+			(xy 104.14 62.23) (xy 104.14 63.5)
+		)
+		(stroke
+			(width 0)
+			(type default)
+		)
+	)
+	(wire
+		(pts
 			(xy 158.75 109.22) (xy 168.91 109.22)
 		)
@@
 	(wire
 		(pts
+			(xy 104.14 62.23) (xy 110.49 62.23)
+		)
+		(stroke
+			(width 0)
+			(type default)
+		)
+	)
+	(wire
+		(pts
 			(xy 120.65 67.31) (xy 120.65 72.39)
 		)
@@
 	(wire
 		(pts
-			(xy 104.14 60.96) (xy 104.14 63.5)
+			(xy 104.14 60.96) (xy 104.14 62.23)
 		)
 		(stroke
@@
 			)
 		)
-		(property "Value" "84R5"
+		(property "Value" "84.5k"
 			(at 106.172 67.056 0)
 			(effects
@@
 			)
 		)
-		(property "LCSC Part #" " C334834"
+		(property "LCSC Part #" "C706195"
 			(at 104.14 66.04 0)
 			(effects
@@
 	)
 	(symbol
-		(lib_id "Connector:TestPoint")
-		(at 186.69 109.22 0)
-		(unit 1)
-		(exclude_from_sim no)
-		(in_bom yes)
-		(on_board yes)
-		(dnp yes)
-		(property "Reference" "TP2"
-			(at 189.23 107.696 0)
-			(effects
-				(font
-					(size 1.27 1.27)
-				)
-				(justify left bottom)
-			)
-		)
-		(property "Value" "TESTPOINT"
-			(at 185.928 106.172 0)
-			(effects
-				(font
-					(size 1.27 1.27)
-				)
-				(justify left bottom)
-				(hide yes)
-			)
-		)
-		(property "Footprint" "TestPoint:TestPoint_Pad_1.0x1.0mm"
-			(at 186.69 109.22 0)
-			(effects
-				(font
-					(size 1.27 1.27)
-				)
-				(hide yes)
-			)
-		)
-		(property "Datasheet" ""
-			(at 186.69 109.22 0)
-			(effects
-				(font
-					(size 1.27 1.27)
-				)
-				(hide yes)
-			)
-		)
-		(property "Description" "SMD test pin"
-			(at 186.69 109.22 0)
-			(effects
-				(font
-					(size 1.27 1.27)
-				)
-				(hide yes)
-			)
-		)
-		(property "LCSC Part #" ""
-			(at 186.69 109.22 0)
-			(effects
-				(font
-					(size 1.27 1.27)
-				)
-				(hide yes)
-			)
-		)
-		(pin "1"
-		)
-		(instances
-			(project "EtherCATControllerLP"
-				(path "/4c927f80-855d-490a-80b2-e5c55283621a/8ad53e1c-08f0-40db-b0fb-703203134f02/386fb4a2-e014-4306-9144-c1ba6edc37f5"
-					(reference "TP2")
-					(unit 1)
-				)
-			)
-		)
-	)
-	(symbol
 		(lib_id "Regulator_Switching:TPS54360DDA")
 		(at 120.65 54.61 0)
@@
 			)
 		)
-		(property "Footprint" "Resistor_SMD:R_0402_1005Metric"
+		(property "Footprint" "Resistor_SMD:R_0603_1608Metric_Pad0.98x0.95mm_HandSolder"
 			(at 104.14 58.42 0)
 			(effects
@@
 			)
 		)
-		(property "LCSC Part #" " C327338"
+		(property "LCSC Part #" "C23076"
 			(at 104.14 58.42 0)
 			(effects
@@
 	)
 	(symbol
+		(lib_id "Connector:TestPoint")
+		(at 158.75 109.22 0)
+		(unit 1)
+		(exclude_from_sim no)
+		(in_bom yes)
+		(on_board yes)
+		(dnp yes)
+		(property "Reference" "TP2"
+			(at 161.29 107.696 0)
+			(effects
+				(font
+					(size 1.27 1.27)
+				)
+				(justify left bottom)
+			)
+		)
+		(property "Value" "TESTPOINT"
+			(at 157.988 106.172 0)
+			(effects
+				(font
+					(size 1.27 1.27)
+				)
+				(justify left bottom)
+				(hide yes)
+			)
+		)
+		(property "Footprint" "TestPoint:TestPoint_Pad_1.0x1.0mm"
+			(at 158.75 109.22 0)
+			(effects
+				(font
+					(size 1.27 1.27)
+				)
+				(hide yes)
+			)
+		)
+		(property "Datasheet" ""
+			(at 158.75 109.22 0)
+			(effects
+				(font
+					(size 1.27 1.27)
+				)
+				(hide yes)
+			)
+		)
+		(property "Description" "SMD test pin"
+			(at 158.75 109.22 0)
+			(effects
+				(font
+					(size 1.27 1.27)
+				)
+				(hide yes)
+			)
+		)
+		(property "LCSC Part #" ""
+			(at 158.75 109.22 0)
+			(effects
+				(font
+					(size 1.27 1.27)
+				)
+				(hide yes)
+			)
+		)
+		(pin "1"
+		)
+		(instances
+			(project "EtherCATControllerHP"
+				(path "/4c927f80-855d-490a-80b2-e5c55283621a/8ad53e1c-08f0-40db-b0fb-703203134f02/386fb4a2-e014-4306-9144-c1ba6edc37f5"
+					(reference "TP2")
+					(unit 1)
+				)
+			)
+		)
+	)
+	(symbol
 		(lib_id "Device:C_Small")
 		(at 92.71 46.99 0)
@@
 		(lib_id "Device:R_Small")
 		(at 100.33 58.42 0)
+		(mirror y)
 		(unit 1)
 		(exclude_from_sim no)
@@
 		(dnp no)
 		(property "Reference" "R1"
-			(at 95.25 57.658 0)
+			(at 105.41 57.658 0)
 			(effects
 				(font
@@
 		)
 		(property "Value" "162K"
-			(at 93.98 59.944 0)
+			(at 106.68 59.944 0)
 			(effects
 				(font
