File: pcb/high-power/EtherCATControllerHP/Temperature.kicad_sch (KiCad schematic)
At the start: 9 parts

Commit message: stash before via stitching
Parts:
- removed C83, C84: 2.2uF, Capacitor_SMD:C_0603_1608Metric, symbol Device:C
- removed R51, R52: 3.3k, Resistor_SMD:R_0603_1608Metric, symbol Device:R
- removed TH2, TH3: 10k, Resistor_SMD:R_0402_1005Metric, symbol Device:Thermistor_NTC
