File: pcb/high-power/EtherCATControllerHP/EtherCATControllerHP.kicad_pcb (KiCad board)
At the start: 2 copper layers, 52 x 52 mm, 0 parts

Commit message: starting HP version
Parts:
- added C1: 10uF, Capacitor_SMD:C_1210_3225Metric, B.Cu at (145.8, 114.8)
- added C10: 10uF, Capacitor_SMD:C_1210_3225Metric, B.Cu at (158.6, 110.2)
- added C12: 4.7uF, Capacitor_SMD:C_1210_3225Metric, B.Cu at (146.4, 106.2)
- added C13: 10pF, Capacitor_SMD:C_0402_1005Metric, B.Cu at (156.4, 80.2)
- added C14: 0.1uF, Capacitor_SMD:C_0402_1005Metric, B.Cu at (144.6, 103.4)
- added C15: 6800pF, Capacitor_SMD:C_0402_1005Metric, B.Cu at (140.0, 97.4)
- added C16: 4.7uF, Capacitor_SMD:C_0805_2012Metric, F.Cu at (166.6, 91.8)
- added C17: 4.7uF, Capacitor_SMD:C_0805_2012Metric, F.Cu at (168.6, 91.8)
- added C18: 39pF, Capacitor_SMD:C_0402_1005Metric, B.Cu at (140.0, 96.2)
- added C19: 0.1uF, Capacitor_SMD:C_0402_1005Metric, B.Cu at (145.4, 100.0)
- added C2: 10uF, Capacitor_SMD:C_1210_3225Metric, B.Cu at (149.0, 114.8)
- added C20: 1uF, Capacitor_SMD:C_0603_1608Metric, B.Cu at (173.2, 103.2)
- added C21: 1uF, Capacitor_SMD:C_0603_1608Metric, B.Cu at (165.0, 113.2)
- added C22: 1uF, Capacitor_SMD:C_0603_1608Metric, B.Cu at (163.4, 111.2)
- added C23: 1uF, Capacitor_SMD:C_0603_1608Metric, B.Cu at (163.4, 108.2)
- added C24: 1uF, Capacitor_SMD:C_0603_1608Metric, B.Cu at (173.0, 105.6)
- added C25: 1uF, Capacitor_SMD:C_0603_1608Metric, B.Cu at (170.0, 102.6)
- added C26: 0.1uF, Capacitor_SMD:C_0805_2012Metric, B.Cu at (173.0, 101.4)
- added C27: 10uF, Capacitor_SMD:CP_Elec_6.3x5.4, F.Cu at (168.4, 108.6)
- added C28: 470pF, Capacitor_SMD:C_0603_1608Metric, B.Cu at (168.2, 113.2)
- added C29: 10uF, Capacitor_SMD:C_0603_1608Metric, B.Cu at (166.6, 113.2)
- added C3: 10uF, Capacitor_SMD:C_1210_3225Metric, B.Cu at (152.2, 114.8)
- added C32: 0.1uF, Capacitor_SMD:C_0603_1608Metric, F.Cu at (95.3, 84.4)
- added C33: 10pF, Capacitor_SMD:C_0402_1005Metric, B.Cu at (160.0, 85.4)
- added C34: 2.2µF, Capacitor_SMD:C_0603_1608Metric, F.Cu at (95.3, 86.9)
- added C35: 2.2µF, Capacitor_SMD:C_0603_1608Metric, F.Cu at (95.3, 89.4)
- added C36: 1uF, Capacitor_SMD:C_0603_1608Metric, F.Cu at (160.6, 93.2)
- added C38: 18pF, Capacitor_SMD:C_0402_1005Metric, F.Cu at (138.4, 91.4)
- added C39: 18pF, Capacitor_SMD:C_0402_1005Metric, F.Cu at (140.8, 86.8)
- added C4: 10uF, Capacitor_SMD:C_1210_3225Metric, B.Cu at (155.4, 114.8)
- added C40: 2.2uF, Capacitor_SMD:C_0603_1608Metric, B.Cu at (171.2, 93.0)
- added C41: 2.2uF, Capacitor_SMD:C_0603_1608Metric, F.Cu at (164.4, 98.8)
- added C42: 0.1uF, Capacitor_SMD:C_0603_1608Metric, B.Cu at (173.2, 99.6)
- added C43: 0.1uF, Capacitor_SMD:C_0603_1608Metric, B.Cu at (171.2, 91.4)
- added C44: 0.1uF, Capacitor_SMD:C_0603_1608Metric, B.Cu at (152.8, 90.2)
- added C45: 0.1uF, Capacitor_SMD:C_0603_1608Metric, B.Cu at (160.4, 102.8)
- added C46: 0.1uF, Capacitor_SMD:C_0603_1608Metric, B.Cu at (162.2, 83.0)
- added C5: 10uF, Capacitor_SMD:C_1210_3225Metric, B.Cu at (158.6, 114.8)
- added C50: 0.1uF, Capacitor_SMD:C_0603_1608Metric, F.Cu at (160.6, 94.8)
- added C51: 1uF, Capacitor_SMD:C_0603_1608Metric, F.Cu at (147.8, 85.8)
- added C52: 1uF, Capacitor_SMD:C_0603_1608Metric, F.Cu at (149.6, 85.8)
- added C53: 0.1uF, Capacitor_SMD:C_0603_1608Metric, F.Cu at (147.2, 101.8)
- added C54: 470pF, Capacitor_SMD:C_0402_1005Metric, F.Cu at (161.2, 97.8)
- added C55: 0.1uF, Capacitor_SMD:C_0603_1608Metric, F.Cu at (160.6, 96.4)
- added C57: 0.1uF, Capacitor_SMD:C_0603_1608Metric, F.Cu at (151.2, 85.8)
- added C58: 0.1uF, Capacitor_SMD:C_0603_1608Metric, F.Cu at (160.6, 91.6)
- added C59: 10pF, Capacitor_SMD:C_0402_1005Metric, F.Cu at (91.9, 46.9)
- added C6: 10uF, Capacitor_SMD:C_1210_3225Metric, B.Cu at (145.8, 110.2)
- added C60: 10pF, Capacitor_SMD:C_0402_1005Metric, F.Cu at (91.9, 48.9)
- added C61: 10pF, Capacitor_SMD:C_0402_1005Metric, F.Cu at (94.8, 43.0)
- added C62: 10nF, Capacitor_SMD:C_1812_4532Metric, B.Cu at (142.0, 114.0)
- added C63: 10pF, Capacitor_SMD:C_0402_1005Metric, F.Cu at (94.8, 44.9)
- added C64: 10pF, Capacitor_SMD:C_0402_1005Metric, F.Cu at (94.8, 46.9)
- added C65: 10pF, Capacitor_SMD:C_0402_1005Metric, F.Cu at (94.8, 48.9)
- added C66: 10pF, Capacitor_SMD:C_0402_1005Metric, F.Cu at (97.6, 43.0)
- added C67: 10pF, Capacitor_SMD:C_0402_1005Metric, F.Cu at (97.6, 44.9)
- added C68: 0.022uF, Capacitor_SMD:C_0402_1005Metric, F.Cu at (97.6, 46.9)
- added C69: 0.022uF, Capacitor_SMD:C_0402_1005Metric, F.Cu at (97.6, 48.9)
- added C7: 10uF, Capacitor_SMD:C_1210_3225Metric, B.Cu at (149.0, 110.2)
- added C70: 0.1uF, Capacitor_SMD:C_0603_1608Metric, F.Cu at (154.4, 85.8)
- added C71: 10nF, Capacitor_SMD:C_0402_1005Metric, F.Cu at (156.2, 84.2)
- added C72: 47uF, Capacitor_SMD:C_0805_2012Metric, B.Cu at (142.8, 98.2)
- added C73: 0.1uF, Capacitor_SMD:C_0603_1608Metric, F.Cu at (152.8, 85.8)
- added C74: 47uF, Capacitor_SMD:C_0805_2012Metric, B.Cu at (142.8, 96.0)
- added C75: 0.1uF, Capacitor_SMD:C_0603_1608Metric, F.Cu at (140.2, 79.0)
- added C76: 1uF, Capacitor_SMD:C_0603_1608Metric, F.Cu at (163.8, 91.6)
- added C77: 0.1uF, Capacitor_SMD:C_0603_1608Metric, F.Cu at (163.8, 90.0)
- added C8: 10uF, Capacitor_SMD:C_1210_3225Metric, B.Cu at (152.2, 110.2)
- added C82: 2.2uF, Capacitor_SMD:C_0603_1608Metric, B.Cu at (158.8, 102.8)
- added C83: 2.2uF, Capacitor_SMD:C_0603_1608Metric, F.Cu at (159.6, 89.6)
- added C84: 2.2uF, Capacitor_SMD:C_0603_1608Metric, B.Cu at (138.6, 90.2)
- added C85: 1uF, Capacitor_SMD:C_0603_1608Metric, F.Cu at (113.0, 77.0)
- added C86: 330pF, Capacitor_SMD:C_0402_1005Metric, F.Cu at (115.4, 66.6)
- added C87: 330pF, Capacitor_SMD:C_0402_1005Metric, F.Cu at (115.4, 68.6)
- added C88: 0.1uF, Capacitor_SMD:C_0603_1608Metric, F.Cu at (109.6, 62.8)
- added C89: 0.1uF, Capacitor_SMD:C_0603_1608Metric, F.Cu at (107.1, 65.3)
- added C9: 10uF, Capacitor_SMD:C_1210_3225Metric, B.Cu at (155.4, 110.2)
- added D1: LTST-C190KGKT, Diode_SMD:D_0603_1608Metric, F.Cu at (143.4, 79.0)
- added D2: B560C, Diode_SMD:D_SMC, B.Cu at (133.4, 100.6)
- added D3: SM24CANB-02HTG, Package_TO_SOT_SMD:SOT-23, F.Cu at (127.2, 101.8)
- added FB1: 2A, 0.05DCR, Inductor_SMD:L_1206_3216Metric, F.Cu at (142.6, 99.8)
- added FB2: 2A, 0.05DCR, Inductor_SMD:L_1206_3216Metric, F.Cu at (144.4, 87.6)
- added FB3: 2A, 0.05DCR, Inductor_SMD:L_1206_3216Metric, F.Cu at (142.6, 97.2)
- added FB4: 2A, 0.05DCR, Inductor_SMD:L_1206_3216Metric, F.Cu at (142.6, 94.6)
- added FB5: 2A, 0.05DCR, Inductor_SMD:L_1206_3216Metric, F.Cu at (163.8, 94.8)
- added H3: MountingHole, MountingHole:MountingHole_2.2mm_M2, F.Cu at (134.0, 84.0)
- added H4: MountingHole, MountingHole:MountingHole_2.2mm_M2, F.Cu at (166.0, 84.0)
- added H5: MountingHole, MountingHole:MountingHole_2.2mm_M2, F.Cu at (134.0, 116.0)
- added H6: MountingHole, MountingHole:MountingHole_2.2mm_M2, F.Cu at (166.0, 116.0)
- added H7: SH_A, MountingHole:MountingHole_2.2mm_M2_Pad, F.Cu at (147.6, 120.0)
- added H8: SH_B, MountingHole:MountingHole_2.2mm_M2_Pad, F.Cu at (160.6, 119.8)
- added H9: SH_C, MountingHole:MountingHole_2.2mm_M2_Pad, F.Cu at (154.2, 120.0)
- added J1: FH41-40S-0.5SH_05_, FH41:HRS_FH41-40S-0.5SH_05_, F.Cu at (132.9, 99.2)
- added J2: Right Angle 1x4, Connector_PinHeader_1.00mm:PinHeader_1x04_P1.00mm_Vertical, F.Cu at (161.1, 79.0)
- added J3: Conn_01x04_Socket, Connector_PinHeader_1.00mm:PinHeader_1x04_P1.00mm_Vertical, F.Cu at (169.4, 86.6)
- added J4: TYPE-C-31-M-12, footprints:HRO_TYPE-C-31-M-12, F.Cu at (150.0, 78.0)
- added J5: UMPT-02-12.5-X-V-S-W-X, UMPT:SAMTEC_UMPT-02-12.5-X-V-S-W-X, F.Cu at (140.5, 113.5)
- added L1: 8.2uH, Inductor_SMD:L_Sunlord_MWSA0603S, B.Cu at (133.8, 107.6)
- added Q1: ~, Package_SO:ONSemi_SO-8FL_488AA, F.Cu at (147.6, 106.9)
- added Q10: ~, Package_SO:ONSemi_SO-8FL_488AA, F.Cu at (160.6, 113.9)
- added Q2: ~, Package_SO:ONSemi_SO-8FL_488AA, F.Cu at (147.6, 114.0)
- added Q5: ~, Package_SO:ONSemi_SO-8FL_488AA, F.Cu at (154.4, 106.9)
- added Q6: ~, Package_SO:ONSemi_SO-8FL_488AA, F.Cu at (154.2, 113.9)
- added Q9: ~, Package_SO:ONSemi_SO-8FL_488AA, F.Cu at (161.2, 106.9)
- added R1: 162K, Resistor_SMD:R_0603_1608Metric, B.Cu at (136.4, 113.1)
- added R11: 5.1K, Resistor_SMD:R_0402_1005Metric, B.Cu at (168.6, 103.0)
- added R12: 5.1K, Resistor_SMD:R_0402_1005Metric, B.Cu at (164.6, 103.0)
- added R13: 5.1K, Resistor_SMD:R_0402_1005Metric, B.Cu at (165.8, 103.0)
- added R14: 5.1K, Resistor_SMD:R_0402_1005Metric, B.Cu at (172.8, 108.2)
- added R15: 2.2R, Resistor_SMD:R_0603_1608Metric, F.Cu at (148.8, 101.8)
- added R16: 2.2R, Resistor_SMD:R_0603_1608Metric, F.Cu at (150.4, 101.8)
- added R17: 2.2R, Resistor_SMD:R_0603_1608Metric, F.Cu at (154.2, 101.8)
- added R18: 2.2R, Resistor_SMD:R_0603_1608Metric, F.Cu at (155.8, 101.8)
- added R2: 523K, Resistor_SMD:R_0402_1005Metric, B.Cu at (139.4, 112.5)
- added R20: 2.2R, Resistor_SMD:R_0603_1608Metric, F.Cu at (163.0, 101.8)
- added R21: 2.2R, Resistor_SMD:R_0603_1608Metric, F.Cu at (159.4, 101.8)
- added R23: 18K, Resistor_SMD:R_0603_1608Metric, F.Cu at (173.4, 103.8)
- added R24: 1k, Resistor_SMD:R_0603_1608Metric, F.Cu at (171.8, 103.8)
- added R25: 1M, Resistor_SMD:R_0402_1005Metric, B.Cu at (139.4, 115.2)
- added R3: 84R5, Resistor_SMD:R_0603_1608Metric, B.Cu at (138.0, 113.1)
- added R31: 10k, Resistor_SMD:R_0603_1608Metric, F.Cu at (157.8, 84.8)
- added R33: 0, Resistor_SMD:R_0402_1005Metric, F.Cu at (139.0, 100.6)
- added R35: 4.7k, Resistor_SMD:R_0402_1005Metric, F.Cu at (138.6, 79.6)
- added R36: 12.1K, Resistor_SMD:R_0402_1005Metric, F.Cu at (145.8, 102.2)
- added R37: 2k, Resistor_SMD:R_0402_1005Metric, F.Cu at (145.8, 84.8)
- added R38: 53.6K, Resistor_SMD:R_0603_1608Metric, B.Cu at (140.4, 94.0)
- added R39: 10.2K, Resistor_SMD:R_0402_1005Metric, B.Cu at (139.0, 94.6)
- added R4: 13K, Resistor_SMD:R_0402_1005Metric, B.Cu at (140.0, 98.6)
- added R41: 22R, Resistor_SMD:R_0603_1608Metric, F.Cu at (162.4, 84.2)
- added R42: 22R, Resistor_SMD:R_0603_1608Metric, F.Cu at (160.8, 84.2)
- added R44: 5.1k, Resistor_SMD:R_0603_1608Metric, B.Cu at (152.0, 79.4)
- added R45: 22R, Resistor_SMD:R_0402_1005Metric, B.Cu at (150.6, 79.0)
- added R46: 22R, Resistor_SMD:R_0402_1005Metric, B.Cu at (149.6, 79.0)
- added R47: 5.1k, Resistor_SMD:R_0603_1608Metric, B.Cu at (148.2, 79.4)
- added R48: 22R, Resistor_SMD:R_0603_1608Metric, F.Cu at (107.1, 67.8)
- added R49: 22R, Resistor_SMD:R_0603_1608Metric, F.Cu at (107.1, 70.3)
- added R5: 1k, Resistor_SMD:R_0603_1608Metric, F.Cu at (141.8, 79.0)
- added R50: 3.3k, Resistor_SMD:R_0603_1608Metric, B.Cu at (157.2, 102.8)
- added R51: 3.3k, Resistor_SMD:R_0603_1608Metric, F.Cu at (159.6, 88.0)
- added R52: 3.3k, Resistor_SMD:R_0603_1608Metric, B.Cu at (138.6, 88.6)
- added R53: 22R, Resistor_SMD:R_0603_1608Metric, F.Cu at (107.1, 72.8)
- added R54: 120R, Resistor_SMD:R_0402_1005Metric, F.Cu at (110.6, 71.2)
- added R55: 0, Resistor_SMD:R_0603_1608Metric, F.Cu at (107.1, 75.3)
- added R56: 0, Resistor_SMD:R_0603_1608Metric, F.Cu at (107.1, 77.8)
- added R6: 500uOhm, Resistor_SMD:R_2512_6332Metric, B.Cu at (152.6, 105.8)
- added R7: 47K, Resistor_SMD:R_0603_1608Metric, F.Cu at (95.3, 91.9)
- added R8: 2k, Resistor_SMD:R_0402_1005Metric, F.Cu at (145.8, 85.8)
- added R9: 0, Resistor_SMD:R_0402_1005Metric, F.Cu at (137.6, 100.6)
- added RN1: 49R9, Resistor_SMD:R_Array_Convex_4x0402, F.Cu at (138.4, 98.3)
- added RN2: 49R9, Resistor_SMD:R_Array_Convex_4x0402, F.Cu at (138.7, 93.0)
- added SW1: EVP-AA202K, footprints:SW_EVP-AA102K_PAN, F.Cu at (157.6, 80.4)
- added TH1: 10k, Resistor_SMD:R_0402_1005Metric, F.Cu at (161.2, 103.0)
- added TH2: 10k, Resistor_SMD:R_0402_1005Metric, F.Cu at (160.0, 86.6)
- added TH3: 10k, Resistor_SMD:R_0402_1005Metric, B.Cu at (138.0, 87.2)
- added TP1: TESTPOINT, TestPoint:TestPoint_Pad_1.0x1.0mm, F.Cu at (62.2, 91.5)
- added TP2: TESTPOINT, TestPoint:TestPoint_Pad_1.0x1.0mm, F.Cu at (95.7, 75.5)
- added TP3: TESTPOINT, TestPoint:TestPoint_Pad_1.0x1.0mm, F.Cu at (95.7, 78.6)
- added TP4: TESTPOINT, TestPoint:TestPoint_Pad_1.0x1.0mm, F.Cu at (62.2, 94.5)
- added U1: STM32F405RGT6, Package_QFP:LQFP-64_10x10mm_P0.5mm, B.Cu at (161.8, 93.4)
- added U2: TPS54360DDAR, Package_SO:TI_SO-PowerPAD-8_ThermalVias, B.Cu at (141.2, 103.4)
- added U3: LDL1117S33R, Package_TO_SOT_SMD:SOT-223, F.Cu at (170.0, 98.4)
- added U4: LAN9252I/ML, footprints:QFN64_ML_MCH, F.Cu at (152.2, 94.6)
- added U5: AS5047P-ATSM, AMS:SOP65P640X120-14N, B.Cu at (150.0, 100.0)
- added U6: MCF8329A1IREER, footprints:WQFN36_REE_TEX, B.Cu at (168.6, 108.2)
- added U7: 24FC512-I/SN, Package_SO:SOP-8_3.9x4.9mm_P1.27mm, F.Cu at (140.6, 83.4)
- added U8: SN65HVD231, Package_SO:SOIC-8_3.9x4.9mm_P1.27mm, B.Cu at (140.6, 83.4)
- added Y1: ABM3B-8.000MHZ-10-1-U-T, Crystal:Crystal_SMD_5032-4Pin_5.0x3.2mm, B.Cu at (158.2, 82.8)
- added Y2: ABM8-25.000MHZ-D2Y-T, Crystal:Crystal_SMD_3225-4Pin_3.2x2.5mm, F.Cu at (139.5, 89.2)
Routing:
- added copper zone on In2.Cu, net 5V
- added copper zone on In2.Cu, net DCBUS
- added copper zone on In2.Cu, net EtherCAT3v3
- added copper zone on In1.Cu, net GND
- added copper zone on In4.Cu, net GND
- added copper zone on In2.Cu, net VCC
Other:
- board size 52 x 52 mm -> 50 x 50 mm
- copper layers 2 -> 6

Commit message: stash before via stitching
Parts:
- removed C71: 10nF, Capacitor_SMD:C_0402_1005Metric
- removed C83, C84: 2.2uF, Capacitor_SMD:C_0603_1608Metric
- removed R31: 10k, Resistor_SMD:R_0603_1608Metric
- removed R45, R46: 22R, Resistor_SMD:R_0402_1005Metric
- removed R51, R52: 3.3k, Resistor_SMD:R_0603_1608Metric
- removed TH2, TH3: 10k, Resistor_SMD:R_0402_1005Metric
- added C11: 1uF, Capacitor_SMD:C_1206_3216Metric, F.Cu at (150.6, 100.9)
- added C30: 1uF, Capacitor_SMD:C_1206_3216Metric, F.Cu at (150.6, 91.9)
- added C31: 330pF, Capacitor_SMD:C_0402_1005Metric, F.Cu at (127.1, 116.0)
- added C37: 0.1uF, Capacitor_SMD:C_0603_1608Metric, B.Cu at (150.1, 80.4)
- added C48: 100uF, 80V, Capacitor_SMD:CP_Elec_10x10, F.Cu at (158.2, 129.2)
- added C49: 0.1uF, Capacitor_SMD:C_0805_2012Metric, F.Cu at (157.4, 102.2)
- added C56: 0.1uF, Capacitor_SMD:C_0805_2012Metric, F.Cu at (159.8, 102.2)
- added C78: 0.1uF, Capacitor_SMD:C_0805_2012Metric, F.Cu at (157.5, 115.0)
- added C79: 0.1uF, Capacitor_SMD:C_0805_2012Metric, F.Cu at (159.8, 115.0)
- added C80: 1uF, Capacitor_SMD:C_1206_3216Metric, F.Cu at (157.2, 97.0)
- added C81: 1uF, Capacitor_SMD:C_1206_3216Metric, F.Cu at (160.0, 97.0)
- added C90: 1uF, Capacitor_SMD:C_1206_3216Metric, F.Cu at (157.2, 89.8)
- added C91: 1uF, Capacitor_SMD:C_1206_3216Metric, F.Cu at (160.0, 89.8)
- added C92: 1uF, Capacitor_SMD:C_1206_3216Metric, F.Cu at (157.3, 110.0)
- added C93: 1uF, Capacitor_SMD:C_1206_3216Metric, F.Cu at (160.0, 110.0)
- added C94: 0.1uF, Capacitor_SMD:C_0805_2012Metric, F.Cu at (157.2, 84.2)
- added C95: 0.1uF, Capacitor_SMD:C_0805_2012Metric, F.Cu at (160.0, 84.2)
- added J6: 2 pin Molex Picoblade, Connector_Molex:Molex_PicoBlade_53048-0210_1x02_P1.25mm_Horizontal, F.Cu at (131.6, 127.1)
- added J7: DEBUG POWER, Connector_PinHeader_1.00mm:PinHeader_1x04_P1.00mm_Vertical, F.Cu at (165.3, 66.7)
- added Q11: ~, Package_SO:ONSemi_SO-8FL_488AA, F.Cu at (177.3, 103.2)
- added Q12: ~, Package_SO:ONSemi_SO-8FL_488AA, F.Cu at (177.3, 109.2)
- added Q3: ~, Package_SO:ONSemi_SO-8FL_488AA, F.Cu at (164.6, 87.4)
- added Q4: ~, Package_SO:ONSemi_SO-8FL_488AA, F.Cu at (170.7, 97.9)
- added Q7: ~, Package_SO:ONSemi_SO-8FL_488AA, F.Cu at (170.7, 112.4)
- added Q8: ~, Package_SO:ONSemi_SO-8FL_488AA, F.Cu at (177.3, 90.8)
- added R10: 22R, Resistor_SMD:R_0402_1005Metric, B.Cu at (149.9, 85.8)
- added R19: 22R, Resistor_SMD:R_0402_1005Metric, B.Cu at (149.9, 84.8)
- C1, C10, C2, C3, C4, C5, C6, C7, C8, C9, R50, U8: moved to F.Cu
- C27: footprint Capacitor_SMD:CP_Elec_6.3x5.4 -> Capacitor_SMD:C_1210_3225Metric; moved to B.Cu
- C32, C34, C35, C38, C39, C50, C54, C59, C60, C61, C63, C64, C65, C66, C67, C75, R15, R16, R17, R18, R20, R21, R23, R24, R35, R37, R41, R42, R7, R8, TP4, U4, U7, Y2: moved to B.Cu
- H3, H4, H5, H6: footprint MountingHole:MountingHole_2.2mm_M2 -> MountingHole:MountingHole_3.2mm_M3_Pad_Via
- J1: value FH41-40S-0.5SH_05_ -> DNP; footprint FH41:HRS_FH41-40S-0.5SH_05_ -> RJ45:BEL_L8AL-1X1T-32A
- J5: value UMPT-02-12.5-X-V-S-W-X -> XT60PW-M; footprint UMPT:SAMTEC_UMPT-02-12.5-X-V-S-W-X -> Connector_AMASS:AMASS_XT60PW-M_1x02_P7.20mm_Horizontal
- R2: footprint Resistor_SMD:R_0402_1005Metric -> Resistor_SMD:R_0603_1608Metric_Pad0.98x0.95mm_HandSolder
- R3: value 84R5 -> 84.5k
- R55, R56: footprint Resistor_SMD:R_0603_1608Metric -> Resistor_SMD:R_0603_1608Metric_Pad0.98x0.95mm_HandSolder
- moved TP1 96.7 mm to (154.1, 121.8)
- moved TP4 85.6 mm to (146.0, 112.0), turned to 180 degrees
- moved C32 74.9 mm to (170.0, 90.0)
- moved C69 71.1 mm to (139.2, 106.6)
- moved C60 69.7 mm to (146.6, 92.1)
- moved C63 67.8 mm to (143.5, 92.1), turned to -90 degrees
- moved R7 67.5 mm to (160.8, 75.4), turned to 90 degrees
- moved TP2 66.5 mm to (162.0, 70.6)
- moved C65 64.9 mm to (142.4, 92.9), turned to -90 degrees
- moved TP3 64.8 mm to (160.0, 70.6)
- moved C34 64.2 mm to (158.6, 97.4), turned to -90 degrees
- moved C68 63.5 mm to (139.2, 94.9)
- moved C61 63.4 mm to (135.1, 91.9), turned to -90 degrees
- moved C59 63.1 mm to (136.1, 91.9), turned to -90 degrees
- moved C88 62.2 mm to (125.2, 123.0)
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Connections:
- H8 pad 1: /SH_C -> /SH_B
- H9 pad 1: /SH_B -> /SH_C
- J1 pad 1: GND -> /ETH1_CT1
- J1 pad 10: GND -> /ETH1_TXN
- J1 pad 11: GND -> /ETH1_TXP
- J1 pad 12: GND -> /ETH0_CT1
- J1 pad 2: GND -> /ETH0_TXN
- J1 pad 3: GND -> /ETH0_TXP
- J1 pad 4: /ETH1_RXN -> /ETH1_RXP
- J1 pad 5: GND -> /ETH1_RXN
- J1 pad 6: /ETH1_RXP -> /ETH0_CT1
- J1 pad 7: GND -> /ETH1_CT1
- J1 pad 8: GND -> /ETH0_RXP
- J1 pad 9: GND -> /ETH0_RXN
- J4 pad B6: Net-(J4-DP2) -> /USB_D+
- J4 pad B7: Net-(J4-DN2) -> /USB_D-
- R12 pad 1: AVCC -> VCC
- R13 pad 1: AVCC -> VCC
- R14 pad 1: AVCC -> VCC
- R2 pad 2: Net-(R2-Pad2) -> Net-(U2-EN)
- R3 pad 1: Net-(R2-Pad2) -> Net-(U2-EN)
- SW1 pad 1: /BOOT0 -> VCC
- SW1 pad 2: unconnected-(SW1-Pad2) -> /BOOT0
- SW1 pad 3: GND -> unconnected-(SW1-Pad3)
- TP2 pad 1: Net-(D1-Pad2) -> VCC
- U1 pad 15: /TEMP_BACKSIDE -> /TEMP_MOSFETS
- U1 pad 16: /TEMP_MOSFETS -> unconnected-(U1-PA2-Pad16)
- U1 pad 17: /TEMP_ICS -> unconnected-(U1-PA3-Pad17)
- U1 pad 2: /SPI2_CS -> /SPI_CS
- U1 pad 25: /IRQ -> unconnected-(U1-PC5-Pad25)
- U1 pad 27: unconnected-(U1-PB1-Pad27) -> /CAN_MODE
- U1 pad 29: /I2C_SDA -> /I2C_SCL
- U1 pad 30: /I2C_SCL -> /I2C_SDA
- U1 pad 41: /SPI_CS -> unconnected-(U1-PA8-Pad41)
- U1 pad 42: unconnected-(U1-PA9-Pad42) -> /IRQ
- U1 pad 43: unconnected-(U1-PA10-Pad43) -> /SPI2_CS
- U1 pad 44: /USB_D- -> Net-(U1-PA11)
- U1 pad 45: /USB_D+ -> Net-(U1-PA12)
- U1 pad 8: /BRAKE -> unconnected-(U1-PC0-Pad8)
- U1 pad 9: /DIR -> unconnected-(U1-PC1-Pad9)
- U2 pad 3: GND -> Net-(U2-EN)
- U6 pad 31: /DIR -> unconnected-(U6-DIR-Pad31)
- U6 pad 34: /BRAKE -> unconnected-(U6-BRAKE-Pad34)
Routing:
- net /Motor/SENSE_P: track 0.00 -> 113.8 mm, vias 0 -> 10
- net AVCC: track 0.00 -> 107.2 mm, vias 0 -> 8
- net 5V: track 0.00 -> 105.8 mm, vias 0 -> 6
- net VCC: track 0.00 -> 100.8 mm, vias 0 -> 21
- net GND: track 0.00 -> 92.0 mm, vias 0 -> 162
- net SHIELD: track 0.00 -> 82.7 mm, vias 0 -> 2
- net /CAN_MODE: track 0.00 -> 77.0 mm, vias 0 -> 2
- net DCBUS: track 0.00 -> 76.9 mm, vias 0 -> 5
- net EtherCAT3v3: track 0.00 -> 52.9 mm, vias 0 -> 16
- net /CAN_TX: track 0.00 -> 45.8 mm, vias 0 -> 2
- net /DRVOFF: track 0.00 -> 45.0 mm, vias 0 -> 2
- net /CAN_RX: track 0.00 -> 43.7 mm, vias 0 -> 2
- net /WAKE: track 0.00 -> 39.1 mm, vias 0 -> 2
- net VDDTXRX2: track 0.00 -> 37.3 mm, vias 0 -> 2
- net /ETH0_TXN: track 0.00 -> 35.1 mm, vias 0 -> 1
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- added copper zone on B.Cu, net /SH_A
- added copper zone on F.Cu, net /SH_A
- added copper zone on B.Cu, net /SH_B
- added copper zone on F.Cu, net /SH_B
- added copper zone on B.Cu, net /SH_C
- added copper zone on F.Cu, net /SH_C
- added copper zone on In2.Cu, net AVCC
- added copper zone on F.Cu, net DCBUS
- added copper zone on B.Cu, net GND
- added copper zone on F.Cu, net GND
- removed copper zone on In2.Cu, net DCBUS
Other:
- board size 50 x 50 mm -> 76 x 76 mm
- board text added: "CANL CANH"

Commit message: finished with HP controller
Parts:
- added G***: LOGO, Stompy:biggerstompy, F.Cu at (122.2, 82.8)
- moved C42 21.1 mm to (148.2, 106.8), turned to 0 degrees
- renumbered TP2 to 3V3, TP3 to 5V, H7 to A, H8 to B, H9 to C
Connections:
- U1 pad 28: GND -> unconnected-(U1-PB2-Pad28)
Routing:
- net GND: track 92.0 -> 121.6 mm, vias 162 -> 472
- net AVCC: track 107.2 -> 122.1 mm, vias 8 -> 6
- net /DRVOFF: track 45.0 -> 48.6 mm
- net /SH_A: track 25.4 -> 28.5 mm, vias 12 -> 14
- net DCBUS: track 76.9 -> 74.0 mm, vias 5 -> 18
- net 5V: track 105.8 -> 103.5 mm
- net Net-(Q10-G): track 29.4 -> 30.8 mm
- net SHIELD: vias 2 -> 1
- net /SH_C: vias 12 -> 13
- added copper zone on B.Cu, net DCBUS
Other:
- board text added: "3V SC G SD"
- board text added: "BOOT0"
- board text added: "DC+"
- board text added: "DC-"
- board text added: "EtherCAT Motor Controller V1"
- board text added: "G 5V AV 3V"
- board text added: "MO MI CK CS"
