File: pcb/high-power/EtherCATControllerHP/Connectors.kicad_sch (KiCad schematic)
At the start: 15 parts, among them J1 FH41-40S-0.5SH_05_, J2 Right Angle 1x4, J3 Conn_01x04_Socket

Commit message: starting HP version
Parts:
- removed H1: DC+ Pin, symbol Mechanical:MountingHole_Pad
- removed H2: DC- Pin, symbol Mechanical:MountingHole_Pad
- removed J1: FH41-40S-0.5SH_05_, FH41-40S-0.5SH_05_:HRS_FH41-40S-0.5SH_05_, symbol FH41-40S-0.5SH_05_:FH41-40S-0.5SH_05_
- removed JP1: Boot Jumper, symbol Jumper:Jumper_2_Open
- removed R31, R32: 22R, Resistor_SMD:R_0603_1608Metric, symbol Device:R
- added C11, C30: 10pF, Capacitor_SMD:C_0402_1005Metric, symbol Device:C
- added C62: 10nF, Capacitor_SMD:C_1812_4532Metric, symbol Device:C
- added C71: 10nF, Capacitor_SMD:C_0402_1005Metric, symbol Device:C
- added J1: DNP, RJ45:BEL_L8AL-1X1T-32A, symbol L8AL-1X1T-32A:L8AL-1X1T-32A
- added J4: TYPE-C-31-M-12, footprints:HRO_TYPE-C-31-M-12, symbol TYPE-C-31-M-12:TYPE-C-31-M-12
- added R25: 1M, Resistor_SMD:R_0402_1005Metric, symbol Device:R
- added R31: 10k, Resistor_SMD:R_0603_1608Metric, symbol Device:R_Small
- added R41, R42: 22R, Resistor_SMD:R_0603_1608Metric, symbol Device:R
- added R44, R47: 5.1k, Resistor_SMD:R_0603_1608Metric, symbol Device:R
- added R45, R46: 22R, Resistor_SMD:R_0402_1005Metric, symbol Device:R
- added SW1: EVP-AA202K, footprints:SW_EVP-AA102K_PAN, symbol 2024-07-26_04-43-59:EVP-AA202K
- H7, H8, H9: footprint (none) -> MountingHole:MountingHole_2.2mm_M2_Pad
- J2: footprint Connector_PinHeader_2.54mm:PinHeader_1x04_P2.54mm_Horizontal -> Connector_PinHeader_1.00mm:PinHeader_1x04_P1.00mm_Vertical; LCSC Part # (none) -> C91552; LCSC Part Number C91552 -> (none); now not fitted
- J3: footprint Hole-Mounts:Nine-Hole -> Connector_PinHeader_1.00mm:PinHeader_1x04_P1.00mm_Vertical; now not fitted
Connections:
- net BOOT0: now also C71.1, R31.2, SW1.1
- net ETH0_CT1: now also C11.2, J1.12 (TRCT1), J1.6 (TRCT2)
- net ETH1_CT1: now also C30.2, J1.1 (TRCT3), J1.7 (TRCT4)
- net GND: now also C11.1, C30.1, C71.2, J1.S1 (SHIELD), J1.S2 (SHIELD), J4.A1_B12 (GND), J4.B1_A12 (GND), R25.2, R44.2, R47.2, SW1.3
- net SHIELD: now also C62.2, J4.S1 (SHIELD), J4.S2 (SHIELD), J4.S3 (SHIELD), J4.S4 (SHIELD)
- net SWCLK: now also R41.2
- net SWDIO: now also R42.1
- net VCC: now also R31.1
- net at J2.1 (Pin_1): now also R42.2
- net at J2.3 (Pin_3): now also R41.1
- new net: J4.A4_B9 (VBUS), J4.B4_A9 (VBUS)
- new net: J4.A5 (CC1), R44.1
- new net: J4.B5 (CC2), R47.1
- new net: J4.B6 (DP2), R46.1
- new net: J4.B7 (DN2), R45.1
- new net: C62.1, R25.1
- new net ETH0_RX_N: J1.10 (TRD1-)
- new net ETH0_RX_P: J1.11 (TRD1+)
- new net ETH0_TX_N: J1.5 (TRD2-)
- new net ETH0_TX_P: J1.4 (TRD2+)
- new net ETH1_RX_N: J1.2 (TRD3-)
- new net ETH1_RX_P: J1.3 (TRD3+)
- new net ETH1_TX_N: J1.9 (TRD4-)
- new net ETH1_TX_P: J1.8 (TRD4+)
- new net USB_D+: J4.A6 (DP1), R46.2
- new net USB_D-: J4.A7 (DN1), R45.2
- no-connect marks 0 -> 5
Other:
- note added: "Belfuse L8AL-1X1T-32A LINK-PP LPJK7436CNL Integrated Magnetics Purchased Separately"
- note added: "ETH1 optional for Line Topology Shared cable with 4 pairs hosts both in and out"
- note added: "SPI (Off-axis Encoder) Padded THT"
- note added: "USB-C"
- note added: "nRESET"
- note removed: "Board to Board Shield FFC 0.5mm pitch Assembled"
- note removed: "SPI (Off-axis Encoder)"
- note removed: "STM32 Boot Jumper"
- moved on the sheet: H7, H8, H9

Commit message: stash before via stitching
Parts:
- removed C11, C30: 10pF, Capacitor_SMD:C_0402_1005Metric, symbol Device:C
- removed C71: 10nF, Capacitor_SMD:C_0402_1005Metric, symbol Device:C
- removed R31: 10k, Resistor_SMD:R_0603_1608Metric, symbol Device:R_Small
- removed R45, R46: 22R, Resistor_SMD:R_0402_1005Metric, symbol Device:R
- added J5: XT60PW-M, Connector_AMASS:AMASS_XT60PW-M_1x02_P7.20mm_Horizontal, symbol 2024-07-02_21-14-47:XT60PW-M
- added J6: 2 pin Molex Picoblade, Connector_Molex:Molex_PicoBlade_53048-0210_1x02_P1.25mm_Horizontal, symbol Connector:Conn_01x02_Pin
- added J7: DEBUG POWER, Connector_PinHeader_1.00mm:PinHeader_1x04_P1.00mm_Vertical, symbol Connector:Conn_01x04_Pin
- H3, H4, H5, H6: footprint MountingHole:MountingHole_2.2mm_M2 -> MountingHole:MountingHole_3.2mm_M3_Pad_Via
Connections:
- net BOOT0: now also SW1.2; no longer SW1.1
- net ETH0_RX_N: now also J1.9 (TRD4-); no longer J1.10 (TRD1-)
- net ETH0_RX_P: now also J1.8 (TRD4+); no longer J1.11 (TRD1+)
- net ETH0_TX_N: now also J1.2 (TRD3-); no longer J1.5 (TRD2-)
- net ETH0_TX_P: now also J1.3 (TRD3+); no longer J1.4 (TRD2+)
- net ETH1_RX_N: now also J1.5 (TRD2-); no longer J1.2 (TRD3-)
- net ETH1_RX_P: now also J1.4 (TRD2+); no longer J1.3 (TRD3+)
- net ETH1_TX_N: now also J1.10 (TRD1-); no longer J1.9 (TRD4-)
- net ETH1_TX_P: now also J1.11 (TRD1+); no longer J1.8 (TRD4+)
- net GND: now also J5.1, J7.1 (Pin_1); no longer J1.S1 (SHIELD), J1.S2 (SHIELD), SW1.3
- net SHIELD: now also J1.S1 (SHIELD), J1.S2 (SHIELD)
- net USB_D+: now also J4.B6 (DP2)
- net USB_D-: now also J4.B7 (DN2)
- net VCC: now also SW1.1, J7.4 (Pin_4)
- new net 5V: J7.2 (Pin_2)
- new net AVCC: J7.3 (Pin_3)
- new net CAN_H: J6.2 (Pin_2)
- new net CAN_L: J6.1 (Pin_1)
- new net DCBUS: J5.2
Other:
- note removed: "nRESET"

Commit message: finished with HP controller
Parts:
- J5: LCSC Part # (none) -> C98732
- R41, R42: LCSC Part # (none) -> C107701
- R44, R47: LCSC Part # (none) -> C706184
- SW1: LCSC Part # (none) -> C79147
Changed lines of the file:
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@@
 			)
 		)
-		(property "LCSC Part #" ""
+		(property "LCSC Part #" "C79147"
 			(at 49.53 120.65 0)
 			(effects
@@
 			)
 		)
+		(property "LCSC Part #" " C706184"
+			(at 118.11 118.11 0)
+			(effects
+				(font
+					(size 1.27 1.27)
+				)
+				(hide yes)
+			)
+		)
 		(pin "2"
 		)
@@
 			)
 		)
+		(property "LCSC Part #" "C98732"
+			(at 43.18 66.04 0)
+			(effects
+				(font
+					(size 1.27 1.27)
+				)
+				(hide yes)
+			)
+		)
 		(pin "2"
 		)
@@
 			)
 		)
+		(property "LCSC Part #" " C706184"
+			(at 185.42 129.54 0)
+			(effects
+				(font
+					(size 1.27 1.27)
+				)
+				(hide yes)
+			)
+		)
 		(pin "2"
 		)
@@
 			)
 		)
+		(property "LCSC Part #" "C107701"
+			(at 124.46 72.39 0)
+			(effects
+				(font
+					(size 1.27 1.27)
+				)
+				(hide yes)
+			)
+		)
 		(pin "1"
 		)
@@
 				(hide yes)
 			)
+		)
+		(property "LCSC Part #" "C107701"
+			(at 124.46 64.77 0)
+			(effects
+				(font
+					(size 1.27 1.27)
+				)
+				(hide yes)
+			)

Commit message: redid layout and mounting
Connections:
- net ETH0_RX_N: now also J1.5 (TRD2-); no longer J1.9 (TRD4-)
- net ETH0_RX_P: now also J1.4 (TRD2+); no longer J1.8 (TRD4+)
- net ETH0_TX_N: now also J1.10 (TRD1-); no longer J1.2 (TRD3-)
- net ETH0_TX_P: now also J1.11 (TRD1+); no longer J1.3 (TRD3+)
- net ETH1_RX_N: now also J1.9 (TRD4-); no longer J1.5 (TRD2-)
- net ETH1_RX_P: now also J1.8 (TRD4+); no longer J1.4 (TRD2+)
- net ETH1_TX_N: now also J1.2 (TRD3-); no longer J1.10 (TRD1-)
- net ETH1_TX_P: now also J1.3 (TRD3+); no longer J1.11 (TRD1+)
Changed lines of the file:
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@@
 		)
 	)
-	(hierarchical_label "ETH1_RX_N"
-		(shape input)
-		(at 242.57 57.15 180)
+	(hierarchical_label "ETH1_TX_P"
+		(shape input)
+		(at 242.57 62.23 180)
 		(fields_autoplaced yes)
 		(effects
@@
 		)
 	)
-	(hierarchical_label "ETH1_TX_N"
-		(shape input)
-		(at 242.57 46.99 180)
+	(hierarchical_label "ETH1_RX_P"
+		(shape input)
+		(at 242.57 72.39 180)
+		(fields_autoplaced yes)
+		(effects
+			(font
+				(size 1.27 1.27)
+			)
+			(justify right)
+		)
+	)
+	(hierarchical_label "ETH0_RX_P"
+		(shape input)
+		(at 242.57 52.07 180)
 		(fields_autoplaced yes)
 		(effects
@@
 		)
 	)
+	(hierarchical_label "ETH1_TX_N"
+		(shape input)
+		(at 242.57 67.31 180)
+		(fields_autoplaced yes)
+		(effects
+			(font
+				(size 1.27 1.27)
+			)
+			(justify right)
+		)
+	)
 	(hierarchical_label "SH_A"
 		(shape input)
@@
 		)
 	)
+	(hierarchical_label "ETH0_CT1"
+		(shape input)
+		(at 217.17 44.45 180)
+		(fields_autoplaced yes)
+		(effects
+			(font
+				(size 1.27 1.27)
+			)
+			(justify right)
+		)
+	)
+	(hierarchical_label "SWCLK"
+		(shape input)
+		(at 116.84 64.77 180)
+		(fields_autoplaced yes)
+		(effects
+			(font
+				(size 1.27 1.27)
+			)
+			(justify right)
+		)
+	)
+	(hierarchical_label "SH_B"
+		(shape input)
+		(at 71.12 34.29 180)
+		(fields_autoplaced yes)
+		(effects
+			(font
+				(size 1.27 1.27)
+			)
+			(justify right)
+		)
+	)
 	(hierarchical_label "ETH0_RX_N"
 		(shape input)
-		(at 242.57 77.47 180)
-		(fields_autoplaced yes)
-		(effects
-			(font
-				(size 1.27 1.27)
-			)
-			(justify right)
-		)
-	)
-	(hierarchical_label "ETH0_CT1"
-		(shape input)
-		(at 217.17 44.45 180)
-		(fields_autoplaced yes)
-		(effects
-			(font
-				(size 1.27 1.27)
-			)
-			(justify right)
-		)
-	)
-	(hierarchical_label "SWCLK"
-		(shape input)
-		(at 116.84 64.77 180)
-		(fields_autoplaced yes)
-		(effects
-			(font
-				(size 1.27 1.27)
-			)
-			(justify right)
-		)
-	)
-	(hierarchical_label "SH_B"
-		(shape input)
-		(at 71.12 34.29 180)
+		(at 242.57 57.15 180)
 		(fields_autoplaced yes)
 		(effects
@@
 		)
 	)
-	(hierarchical_label "ETH1_TX_P"
+	(hierarchical_label "SPI_MOSI"
+		(shape input)
+		(at 118.11 45.72 180)
+		(fields_autoplaced yes)
+		(effects
+			(font
+				(size 1.27 1.27)
+			)
+			(justify right)
+		)
+	)
+	(hierarchical_label "ETH1_CT1"
+		(shape input)
+		(at 217.17 64.77 180)
+		(fields_autoplaced yes)
+		(effects
+			(font
+				(size 1.27 1.27)
+			)
+			(justify right)
+		)
+	)
+	(hierarchical_label "SPI_MISO"
+		(shape input)
+		(at 118.11 43.18 180)
+		(fields_autoplaced yes)
+		(effects
+			(font
+				(size 1.27 1.27)
+			)
+			(justify right)
+		)
+	)
+	(hierarchical_label "ETH0_TX_N"
+		(shape input)
+		(at 242.57 46.99 180)
+		(fields_autoplaced yes)
+		(effects
+			(font
+				(size 1.27 1.27)
+			)
+			(justify right)
+		)
+	)
+	(hierarchical_label "BOOT0"
+		(shape input)
+		(at 49.53 128.27 180)
+		(fields_autoplaced yes)
+		(effects
+			(font
+				(size 1.27 1.27)
+			)
+			(justify right)
+		)
+	)
+	(hierarchical_label "ETH0_TX_P"
 		(shape input)
 		(at 242.57 41.91 180)
-		(fields_autoplaced yes)
-		(effects
-			(font
-				(size 1.27 1.27)
-			)
-			(justify right)
-		)
-	)
-	(hierarchical_label "ETH0_RX_P"
-		(shape input)
-		(at 242.57 72.39 180)
-		(fields_autoplaced yes)
-		(effects
-			(font
-				(size 1.27 1.27)
-			)
-			(justify right)
-		)
-	)
-	(hierarchical_label "ETH0_TX_N"
-		(shape input)
-		(at 242.57 67.31 180)
-		(fields_autoplaced yes)
-		(effects
-			(font
-				(size 1.27 1.27)
-			)
-			(justify right)
-		)
-	)
-	(hierarchical_label "ETH1_RX_P"
-		(shape input)
-		(at 242.57 52.07 180)
-		(fields_autoplaced yes)
-		(effects
-			(font
-				(size 1.27 1.27)
-			)
-			(justify right)
-		)
-	)
-	(hierarchical_label "SPI_MOSI"
-		(shape input)
-		(at 118.11 45.72 180)
-		(fields_autoplaced yes)
-		(effects
-			(font
-				(size 1.27 1.27)
-			)
-			(justify right)
-		)
-	)
-	(hierarchical_label "ETH1_CT1"
-		(shape input)
-		(at 217.17 64.77 180)
-		(fields_autoplaced yes)
-		(effects
-			(font
-				(size 1.27 1.27)
-			)
-			(justify right)
-		)
-	)
-	(hierarchical_label "SPI_MISO"
-		(shape input)
-		(at 118.11 43.18 180)
-		(fields_autoplaced yes)
-		(effects
-			(font
-				(size 1.27 1.27)
-			)
-			(justify right)
-		)
-	)
-	(hierarchical_label "BOOT0"
-		(shape input)
-		(at 49.53 128.27 180)
 		(fields_autoplaced yes)
 		(effects
@@
 		)
 	)
-	(hierarchical_label "ETH0_TX_P"
-		(shape input)
-		(at 242.57 62.23 180)
-		(fields_autoplaced yes)
-		(effects
+	(hierarchical_label "ETH1_RX_N"
+		(shape input)
+		(at 242.57 77.47 180)
+		(fields_autoplaced yes)
+		(effects
