File: pcb/high-power/EtherCATControllerHP/MOSFETs.kicad_sch (KiCad schematic)
At the start: 19 parts

Commit message: starting HP version
Parts:
- removed Q11, Q12, Q3, Q4, Q7, Q8: ~, DFN_2NLT1G_ONS, symbol 2024-07-02_05-47-45:NTMFS5C612NLT1G
- Q1: footprint DFN_2NLT1G_ONS -> Package_SO:ONSemi_SO-8FL_488AA; LCSC Part # (none) -> C348543; LCSC Part Number C348543 -> (none)
- Q10, Q2, Q5, Q6, Q9: footprint DFN_2NLT1G_ONS -> Package_SO:ONSemi_SO-8FL_488AA
- R15, R16, R17, R18, R20, R21: LCSC Part # (none) -> C112307
- R6: LCSC Part # (none) -> C500733
Other:
- note added: "MOSFETS: NTMFS5C612NLT1G 60V, 36A Ta Downsized for low-power variant"
- note removed: "MOSFETS: NTMFS5C612NLT1G 60V, 36A Ta"
- moved on the sheet: Q1, Q10, Q2, Q5, Q6, Q9

Commit message: stash before via stitching
Parts:
- added Q11, Q12, Q3, Q4, Q7, Q8: ~, Package_SO:ONSemi_SO-8FL_488AA, symbol 2024-07-02_05-47-45:NTMFS5C612NLT1G
Connections:
- net DCBUS: now also Q3.5 (D), Q4.5 (D), Q7.5 (D)
- net SENSE_P: now also Q11.1 (S), Q11.2 (S), Q11.3 (S), Q12.1 (S), Q12.2 (S), Q12.3 (S), Q8.1 (S), Q8.2 (S), Q8.3 (S)
- net SH_A: now also Q3.1 (S), Q3.2 (S), Q3.3 (S), Q8.5 (D)
- net SH_B: now also Q11.5 (D), Q4.1 (S), Q4.2 (S), Q4.3 (S)
- net SH_C: now also Q12.5 (D), Q7.1 (S), Q7.2 (S), Q7.3 (S)
- net at Q1.4 (G), R15.1: now also Q3.4 (G)
- net at Q10.4 (G), R21.2: now also Q12.4 (G)
- net at Q9.4 (G), R20.1: now also Q7.4 (G)
- net at Q5.4 (G), R18.1: now also Q4.4 (G)
- net at Q2.4 (G), R16.2: now also Q8.4 (G)
- net at Q6.4 (G), R17.1: now also Q11.4 (G)

Commit message: finished with HP controller
Parts:
- Q10, Q2, Q5, Q6, Q9: LCSC Part # (none) -> C348543
Changed lines of the file:
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@@
 			)
 		)
+		(property "LCSC Part #" "C348543"
+			(at 123.19 71.12 0)
+			(effects
+				(font
+					(size 1.27 1.27)
+				)
+				(hide yes)
+			)
+		)
 		(pin "1"
 		)
@@
 			)
 		)
+		(property "LCSC Part #" "C348543"
+			(at 123.19 96.52 0)
+			(effects
+				(font
+					(size 1.27 1.27)
+				)
+				(hide yes)
+			)
+		)
 		(pin "5"
 		)
@@
 			)
 		)
+		(property "LCSC Part #" "C348543"
+			(at 168.91 71.12 0)
+			(effects
+				(font
+					(size 1.27 1.27)
+				)
+				(hide yes)
+			)
+		)
 		(pin "5"
 		)
@@
 			)
 		)
+		(property "LCSC Part #" "C348543"
+			(at 168.91 96.52 0)
+			(effects
+				(font
+					(size 1.27 1.27)
+				)
+				(hide yes)
+			)
+		)
 		(pin "4"
 		)
@@
 			)
 		)
-		(property "LCSC Part #" ""
+		(property "LCSC Part #" "C348543"
 			(at 77.47 96.52 0)
 			(effects

Commit message: redid layout and mounting
Parts:
- added NT1, NT2: NetTie_2, NetTie:NetTie-2_SMD_Pad2.0mm, symbol Device:NetTie_2
Connections:
- net GND: now also NT1.1
- net SENSE_P: now also NT2.2; no longer Q10.1 (S), Q10.2 (S), Q10.3 (S), Q11.1 (S), Q11.2 (S), Q11.3 (S), Q12.1 (S), Q12.2 (S), Q12.3 (S), Q2.1 (S), Q2.2 (S), Q2.3 (S), Q6.1 (S), Q6.2 (S), Q6.3 (S), Q8.1 (S), Q8.2 (S), Q8.3 (S), R6.1
- new net LSS: NT2.1, Q10.1 (S), Q10.2 (S), Q10.3 (S), Q11.1 (S), Q11.2 (S), Q11.3 (S), Q12.1 (S), Q12.2 (S), Q12.3 (S), Q2.1 (S), Q2.2 (S), Q2.3 (S), Q6.1 (S), Q6.2 (S), Q6.3 (S), Q8.1 (S), Q8.2 (S), Q8.3 (S), R6.1
- new net SENSE_N: NT1.2
Changed lines of the file:
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@@
 	)
 	(junction
+		(at 172.72 137.16)
+		(diameter 0)
+		(color 0 0 0 0)
+	)
+	(junction
 		(at 179.07 76.2)
 		(diameter 0)
@@
 	)
 	(junction
-		(at 162.56 137.16)
+		(at 176.53 129.54)
 		(diameter 0)
 		(color 0 0 0 0)
@@
 	(wire
 		(pts
-			(xy 176.53 101.6) (xy 176.53 137.16)
+			(xy 176.53 101.6) (xy 176.53 129.54)
 		)
 		(stroke
@@
 	(wire
 		(pts
+			(xy 176.53 129.54) (xy 176.53 137.16)
+		)
+		(stroke
+			(width 0)
+			(type default)
+		)
+	)
+	(wire
+		(pts
 			(xy 151.13 55.88) (xy 161.29 55.88)
 		)
@@
 	(wire
 		(pts
-			(xy 130.81 137.16) (xy 162.56 137.16)
+			(xy 130.81 137.16) (xy 172.72 137.16)
 		)
 		(stroke
@@
 	(wire
 		(pts
-			(xy 162.56 137.16) (xy 176.53 137.16)
+			(xy 85.09 45.72) (xy 97.79 45.72)
 		)
 		(stroke
@@
 	(wire
 		(pts
-			(xy 85.09 45.72) (xy 97.79 45.72)
+			(xy 151.13 111.76) (xy 161.29 111.76)
 		)
 		(stroke
@@
 	(wire
 		(pts
-			(xy 151.13 111.76) (xy 161.29 111.76)
+			(xy 172.72 137.16) (xy 176.53 137.16)
 		)
 		(stroke
@@
 	(wire
 		(pts
+			(xy 181.61 129.54) (xy 176.53 129.54)
+		)
+		(stroke
+			(width 0)
+			(type default)
+		)
+	)
+	(wire
+		(pts
 			(xy 176.53 76.2) (xy 176.53 86.36)
 		)
@@
 		)
 	)
+	(hierarchical_label "LSS"
+		(shape input)
+		(at 181.61 129.54 0)
+		(fields_autoplaced yes)
+		(effects
+			(font
+				(size 1.27 1.27)
+			)
+			(justify left)
+		)
+	)
 	(hierarchical_label "GH_B"
 		(shape input)
@@
 		)
 	)
+	(hierarchical_label "SENSE_N"
+		(shape output)
+		(at 152.4 153.67 0)
+		(fields_autoplaced yes)
+		(effects
+			(font
+				(size 1.27 1.27)
+			)
+			(justify left)
+		)
+	)
+	(hierarchical_label "SENSE_P"
+		(shape output)
+		(at 152.4 140.97 0)
+		(fields_autoplaced yes)
+		(effects
+			(font
+				(size 1.27 1.27)
+			)
+			(justify left)
+		)
+	)
 	(hierarchical_label "GL_A"
 		(shape input)
@@
 		)
 	)
-	(hierarchical_label "SENSE_N"
-		(shape output)
-		(at 147.32 153.67 0)
-		(fields_autoplaced yes)
-		(effects
-			(font
-				(size 1.27 1.27)
-			)
-			(justify left)
-		)
-	)
-	(hierarchical_label "SENSE_P"
-		(shape output)
-		(at 147.32 140.97 0)
-		(fields_autoplaced yes)
-		(effects
-			(font
-				(size 1.27 1.27)
-			)
-			(justify left)
-		)
-	)
 	(symbol
 		(lib_name "NTMFS5C612NLT1G_3")
@@
 	)
 	(symbol
+		(lib_id "Device:NetTie_2")
+		(at 149.86 153.67 0)
+		(unit 1)
+		(exclude_from_sim no)
+		(in_bom no)
+		(on_board yes)
+		(dnp no)
+		(fields_autoplaced yes)
+		(property "Reference" "NT1"
+			(at 149.86 148.59 0)
+			(effects
+				(font
+					(size 1.27 1.27)
+				)
+			)
+		)
+		(property "Value" "NetTie_2"
+			(at 149.86 151.13 0)
+			(effects
+				(font
+					(size 1.27 1.27)
+				)
+			)
+		)
+		(property "Footprint" "NetTie:NetTie-2_SMD_Pad2.0mm"
+			(at 149.86 153.67 0)
+			(effects
+				(font
+					(size 1.27 1.27)
+				)
+				(hide yes)
+			)
+		)
+		(property "Datasheet" "~"
+			(at 149.86 153.67 0)
+			(effects
+				(font
+					(size 1.27 1.27)
+				)
+				(hide yes)
+			)
+		)
+		(property "Description" "Net tie, 2 pins"
+			(at 149.86 153.67 0)
+			(effects
+				(font
+					(size 1.27 1.27)
+				)
+				(hide yes)
+			)
+		)
+		(pin "1"
+		)
+		(pin "2"
+		)
+		(instances
+			(project ""
+				(path "/4c927f80-855d-490a-80b2-e5c55283621a/b8886fcf-711b-4283-9745-a57e39aa3085/55580437-8668-4251-b652-b45caec55db3"
+					(reference "NT1")
+					(unit 1)
+				)
+			)
+		)
+	)
+	(symbol
 		(lib_id "Device:R")
 		(at 118.11 111.76 270)
@@
 	(symbol
 		(lib_id "power:PWR_FLAG")
-		(at 162.56 137.16 180)
+		(at 172.72 137.16 180)
 		(unit 1)
 		(exclude_from_sim no)
@@
 		(fields_autoplaced yes)
 		(property "Reference" "#FLG011"
-			(at 162.56 139.065 0)
+			(at 172.72 139.065 0)
 			(effects
 				(font
@@
 		)
 		(property "Value" "PWR_FLAG"
-			(at 162.56 142.24 0)
+			(at 172.72 142.24 0)
 			(effects
 				(font
@@
 		)
 		(property "Footprint" ""
-			(at 162.56 137.16 0)
+			(at 172.72 137.16 0)
 			(effects
 				(font
@@
 		)
 		(property "Datasheet" "~"
-			(at 162.56 137.16 0)
+			(at 172.72 137.16 0)
 			(effects
 				(font
@@
 		)
 		(property "Description" "Special symbol for telling ERC where power comes from"
-			(at 162.56 137.16 0)
+			(at 172.72 137.16 0)
 			(effects
 				(font
@@
 					(unit 1)
 				)
+			)
+		)
+	)
+	(symbol
+		(lib_id "Device:NetTie_2")
+		(at 149.86 140.97 0)
+		(unit 1)
+		(exclude_from_sim no)
+		(in_bom no)
+		(on_board yes)
+		(dnp no)
+		(fields_autoplaced yes)
+		(property "Reference" "NT2"
+			(at 149.86 135.89 0)
+			(effects
+				(font
+					(size 1.27 1.27)
+				)
+			)
+		)
+		(property "Value" "NetTie_2"
+			(at 149.86 138.43 0)
+			(effects
+				(font
+					(size 1.27 1.27)
+				)
+			)
+		)
+		(property "Footprint" "NetTie:NetTie-2_SMD_Pad2.0mm"
+			(at 149.86 140.97 0)
+			(effects
+				(font
+					(size 1.27 1.27)
+				)
+				(hide yes)
+			)
+		)
+		(property "Datasheet" "~"
+			(at 149.86 140.97 0)
+			(effects
+				(font
+					(size 1.27 1.27)
+				)
+				(hide yes)
+			)
+		)
+		(property "Description" "Net tie, 2 pins"
+			(at 149.86 140.97 0)
+			(effects
+				(font
+					(size 1.27 1.27)
+				)
+				(hide yes)
+			)
+		)
+		(pin "1"
+		)
+		(pin "2"
+		)
+		(instances
+			(project "EtherCATControllerHP"
+				(path "/4c927f80-855d-490a-80b2-e5c55283621a/b8886fcf-711b-4283-9745-a57e39aa3085/55580437-8668-4251-b652-b45caec55db3"
+					(reference "NT2")
+					(unit 1)
+				)
