File: pcb/high-power/EtherCATControllerHP/Motor.kicad_sch (KiCad schematic)
At the start: 15 parts, among them U6 MCF8329A1IREER

Commit message: starting HP version
Parts:
- C20, C21, C22, C23, C25: footprint (none) -> Capacitor_SMD:C_0603_1608Metric; LCSC Part # (none) -> C106858
- C24: value C_Small -> 1uF; footprint (none) -> Capacitor_SMD:C_0603_1608Metric; LCSC Part # (none) -> C106858
- C26: footprint (none) -> Capacitor_SMD:C_0805_2012Metric; LCSC Part # (none) -> C28233
- C27: footprint (none) -> Capacitor_SMD:CP_Elec_6.3x5.4; LCSC Part # (none) -> C2977481
- C28: footprint (none) -> Capacitor_SMD:C_0603_1608Metric; LCSC Part # (none) -> C107062
- C29: footprint (none) -> Capacitor_SMD:C_0603_1608Metric; LCSC Part # (none) -> C194427
- R11, R12, R13, R14: footprint (none) -> Resistor_SMD:R_0402_1005Metric; LCSC Part # (none) -> C105872
- U6: footprint WQFN36_REE_TEX -> footprints:WQFN36_REE_TEX; LCSC Part # (none) -> C22399784; LCSC Part Number C22399784 -> (none)
Other:
- note removed: "Bulk Cap"

Commit message: stash before via stitching
Parts:
- removed C27: 10uF, Capacitor_SMD:CP_Elec_6.3x5.4, symbol Device:C_Polarized_Small
- added C27: 10uF, Capacitor_SMD:C_1210_3225Metric, symbol Device:C
Connections:
- net AVCC: no longer R12.1, R13.1, R14.1
- net DCBUS: now also C27.1
- net GND: now also C27.2
- net BRAKE: no longer names the net of U6.34 (BRAKE)
- net DIR: no longer names the net of U6.31 (DIR)
- new net VCC: R12.1, R13.1, R14.1
- no-connect marks 3 -> 5

Commit message: redid layout and mounting
Parts:
- C21, C22, C23: LCSC Part # C106858 -> C105174
Connections:
- net AVCC: now also R12.1, R13.1
- net SENSE_P: no longer U6.21 (LSS)
- net VCC: no longer R12.1, R13.1
- new net LSS: U6.21 (LSS)
Other:
- sheet MOSFETs ports: added LSS; removed none
Changed lines of the file:
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@@
 	(wire
 		(pts
+			(xy 193.04 55.88) (xy 193.04 58.42)
+		)
+		(stroke
+			(width 0)
+			(type default)
+		)
+	)
+	(wire
+		(pts
 			(xy 207.01 100.33) (xy 209.55 100.33)
 		)
@@
 		)
 	)
-	(label "SENSE_P"
+	(label "LSS"
 		(at 157.48 113.03 0)
 		(fields_autoplaced yes)
@@
 		)
 	)
+	(label "LSS"
+		(at 238.76 83.82 0)
+		(fields_autoplaced yes)
+		(effects
+			(font
+				(size 1.27 1.27)
+			)
+			(justify left bottom)
+		)
+	)
 	(label "SH_C"
 		(at 241.3 100.33 0)
@@
 	(symbol
 		(lib_id "power:VCC")
-		(at 193.04 58.42 0)
+		(at 193.04 55.88 0)
 		(unit 1)
 		(exclude_from_sim no)
@@
 		(fields_autoplaced yes)
 		(property "Reference" "#PWR032"
-			(at 193.04 62.23 0)
+			(at 193.04 59.69 0)
 			(effects
 				(font
@@
 			)
 		)
-		(property "Value" "VCC"
-			(at 193.04 53.34 0)
+		(property "Value" "AVCC"
+			(at 195.58 54.6099 0)
 			(effects
 				(font
 					(size 1.27 1.27)
 				)
+				(justify left)
 			)
 		)
 		(property "Footprint" ""
-			(at 193.04 58.42 0)
+			(at 193.04 55.88 0)
 			(effects
 				(font
@@
 		)
 		(property "Datasheet" ""
-			(at 193.04 58.42 0)
+			(at 193.04 55.88 0)
 			(effects
 				(font
@@
 		)
 		(property "Description" "Power symbol creates a global label with name \"VCC\""
-			(at 193.04 58.42 0)
+			(at 193.04 55.88 0)
 			(effects
 				(font
@@
 			)
 		)
-		(property "LCSC Part #" "C106858"
+		(property "LCSC Part #" "C105174"
 			(at 58.42 101.6 0)
 			(effects
@@
 			)
 		)
-		(property "LCSC Part #" "C106858"
+		(property "LCSC Part #" "C105174"
 			(at 58.42 111.76 0)
 			(effects
@@
 			)
 		)
-		(property "LCSC Part #" "C106858"
+		(property "LCSC Part #" "C105174"
 			(at 58.42 91.44 0)
 			(effects
@@
 			(effects
 				(font
+					(size 1.27 1.27)
+				)
+				(justify right)
+			)
+		)
+		(pin "LSS" input
+			(at 238.76 83.82 0)
+			(effects
+				(font
