File: pcb/high-power/EtherCATControllerHP/Power.kicad_sch (KiCad schematic)
At the start: 60 parts, among them U2 TPS54360DDAR, U3 LDL1117S33R, U4 LP5907MFX-3.3_NOPB, U8 LM76005RNPR

Commit message: starting HP version
Parts:
- removed C13, C14, C80: 2.2uF, symbol Device:C_Small
- removed C15: 39pF, symbol Device:C_Small
- removed C16, C17, C18: 4.7uF, Capacitor_SMD:C_0805_2012Metric, symbol Device:C
- removed C37, C38, C39, C55, C56, C57: 0.1uF, symbol Device:C
- removed C74: 6800pF, symbol Device:C_Small
- removed C75: 0.1uF, symbol Device:C_Small
- removed C77: 47uF, symbol Device:C_Small
- removed C78: 4.7pF, symbol Device:C_Small
- removed C79, C81, C83: 470nF, symbol Device:C_Small
- removed C82: 150uF, symbol Device:C_Small
- removed D1: LTST-C190KGKT, Diode_SMD:D_0603_1608Metric, symbol LTST-C190KGKT:LTST-C190KGKT
- removed D2: B560C, symbol Device:D_Schottky
- removed L1: 8.2uH, symbol Device:L_Small
- removed L2: 5.6uH, symbol Device:L_Small
- removed R1: 523K, symbol Device:R_Small
- removed R2: 162K, symbol Device:R_Small
- removed R3: 84.5, symbol Device:R_Small
- removed R38: 53.6K, symbol Device:R_Small
- removed R39: 10.2K, symbol Device:R_Small
- removed R4: 13K, symbol Device:R_Small
- removed R40: 100k, symbol Device:R_Small
- removed R41: 100K, symbol Device:R_Small
- removed R42: 43.2K, symbol Device:R_Small
- removed R5: 1k, Resistor_SMD:R_0603_1608Metric, symbol Device:R
- removed TP2, TP3, TP5: TESTPOINT, TestPoint:TestPoint_Pad_1.0x1.0mm, symbol Connector:TestPoint
- removed U2: TPS54360DDAR, Package_SO:TI_SO-PowerPAD-8_ThermalVias, symbol Regulator_Switching:TPS54360DDA
- removed U3: LDL1117S33R, Package_TO_SOT_SMD:SOT-223, symbol LDL1117S33R:LDL1117S33R
- removed U4: LP5907MFX-3.3_NOPB, Package_TO_SOT_SMD:SOT-23-5, symbol LP5907MFX-3.3_NOPB:LP5907MFX-3.3_NOPB
- removed U8: LM76005RNPR, RNP0030A, symbol 2024-07-02_05-34-37:LM76005RNPR
- added C10, C5, C6, C9: 10uF, Capacitor_SMD:C_1210_3225Metric, symbol Device:C
- added C77: ${CAPACITANCE}, Capacitor_SMD:C_0603_1608Metric, symbol Device:C
- added FB5: 2A, 0.05DCR, Inductor_SMD:L_1206_3216Metric, symbol Device:FerriteBead_Small
- C1, C2, C3, C4: footprint (none) -> Capacitor_SMD:C_1210_3225Metric; LCSC Part # (none) -> C5156756; LCSC Part Number C153035 -> (none)
- C40: LCSC Part # (none) -> C77183
- C41: value ${CAPACITANCE} -> 2.2uF; LCSC Part # (none) -> C77183
- C42: LCSC Part # (none) -> C14663
- C43, C44, C45, C46: LCSC Part # (none) -> C77055
- C7, C8: value 22uF -> 10uF; footprint (none) -> Capacitor_SMD:C_1210_3225Metric; LCSC Part # (none) -> C5156756; LCSC Part Number C1921234 -> (none)
- C76: value 47uF -> 1uF; footprint (none) -> Capacitor_SMD:C_0603_1608Metric; LCSC Part # (none) -> C106858
- R23: LCSC Part # (none) -> C98220
- R24: LCSC Part # (none) -> C22548
- TP1, TP4: now not fitted
Connections:
- net 5V: no longer C76.1
- net AVCC: no longer TP1.1
- net DCBUS: now also TP1.1, C10.1, C5.1, C6.1, C9.1
- net EtherCAT3v3: now also C76.1, C77.1, FB5.2
- net GND: now also C10.2, C5.2, C6.2, C77.2, C9.2
- net VCC: now also FB5.1
- no-connect marks 9 -> 0
Other:
- added sheet Regulators (Regulators.kicad_sch)
- note added: "AVCC supplied by MCF8329A"
- note removed: "5V out"
- note removed: "Analog 3v3"
- note removed: "Digital 3v3"
- note removed: "EtherCAT 3v3"
- moved on the sheet: C1, C40, C41, C42, C43, C44, C45, C46, R23, R24

Commit message: stash before via stitching
Parts:
- added C11, C30, C80, C81, C90, C91, C92, C93: 1uF, Capacitor_SMD:C_1206_3216Metric, symbol Device:C
- added C37: ${CAPACITANCE}, Capacitor_SMD:C_0603_1608Metric, symbol Device:C
- added C48: 100uF, 80V, Capacitor_SMD:CP_Elec_10x10, symbol Device:C_Polarized
- added C49, C56, C78, C79, C94, C95: 0.1uF, Capacitor_SMD:C_0805_2012Metric, symbol Device:C_Small
Connections:
- net DCBUS: now also C11.1, C30.1, C48.1, C49.1, C56.1, C78.1, C79.1, C80.1, C81.1, C90.1, C91.1, C92.1, C93.1, C94.1, C95.1
- net GND: now also C11.2, C30.2, C37.2, C48.2, C49.2, C56.2, C78.2, C79.2, C80.2, C81.2, C90.2, C91.2, C92.2, C93.2, C94.2, C95.2
- net VCC: now also C37.1
Other:
- note added: "10uF bypasses 4x bulk caps"
- note removed: "22uF Stacked Ceramic Bypass 10uF bypasses Bulk Caps on IO Board"
- moved on the sheet: C40, C41, C42, C43, C44, C45, C46, C76, C77, FB5, R23, R24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

Commit message: redid layout and mounting
Parts:
- removed C10, C4, C9: 10uF, Capacitor_SMD:C_1210_3225Metric, symbol Device:C
- removed C30, C81, C92, C93: 1uF, Capacitor_SMD:C_1206_3216Metric, symbol Device:C
- removed TP4: TESTPOINT, TestPoint:TestPoint_Pad_1.0x1.0mm, symbol Connector:TestPoint
- added C47: 100uF, 80V, Capacitor_SMD:CP_Elec_10x10, symbol Device:C_Polarized
Connections:
- net DCBUS: now also C47.1
- net GND: now also C47.2
Other:
- moved on the sheet: C11, C5, C6, C80, C90, C91, TP1
