File: pcb/high-power/EtherCATControllerHP/Encoders.kicad_sch (KiCad schematic)
At the start: 8 parts, among them U5 AS5047P-ATSM

Commit message: starting HP version
Parts:
- removed C47, C48, C49: 22nF, Capacitor_SMD:C_0402_1005Metric, symbol Device:C
- removed R27, R28, R29: 3.3k, Resistor_SMD:R_0603_1608Metric, symbol Device:R
- C19: value 100nF -> 0.1uF; LCSC Part # (none) -> C77055
- U5: LCSC Part # (none) -> C962063; LCSC Part Number C962063 -> (none)
Connections:
- net ENC_A: no longer names the net of U5.7 (A)
- net ENC_B: no longer names the net of U5.6 (B)
- net ENC_Z: no longer names the net of U5.14 (I/PWM)
- no-connect marks 3 -> 6
Other:
- moved on the sheet: C19, U5

Commit message: fixed bom
Parts:
- C19: LCSC Part # C77055 -> C513772
Changed lines of the file:
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@@
 			)
 		)
-		(property "LCSC Part #" "C77055"
+		(property "LCSC Part #" "C513772"
 			(at 139.7 44.45 0)
 			(effects
